Commit message: changed arm links reference frames and joint names

File: doris_arm_description/urdf/doris_arm_description.urdf (robot description, URDF)
Before this commit: robot doris_arm_description, 9 links, 8 joints
Links:
- removed link arm_link
- removed link gripper_left
- removed link gripper_right
- removed link pitch_link
- added link elbow_link, mass 0.0892046248471317; collision mesh filename=package://doris_arm_description/meshes/elbow_link.STL; visual mesh filename=package://doris_arm_description/meshes/elbow_link.STL
- added link gripper_link, mass 0.0174078384350788; collision mesh filename=package://doris_arm_description/meshes/gripper_link.STL; visual mesh filename=package://doris_arm_description/meshes/gripper_link.STL
- added link left_finger_link, mass 0.0083226; collision mesh filename=package://doris_arm_description/meshes/left_finger_link.STL; visual mesh filename=package://doris_arm_description/meshes/left_finger_link.STL
- added link right_finger_link, mass 0.00832263335631547; collision mesh filename=package://doris_arm_description/meshes/right_finger_link.STL; visual mesh filename=package://doris_arm_description/meshes/right_finger_link.STL
- added link roll_2_link, mass 0.15161780969895; collision mesh filename=package://doris_arm_description/meshes/roll_2_link.STL; visual mesh filename=package://doris_arm_description/meshes/roll_2_link.STL
- link forearm_link: mass 0.073149 -> 0.0731491894717436
- link roll_link: mass 0.034548 -> 0.108644948048519
- link shoulder_link: mass 0.18737 -> 0.187371975468428
- link yaw_link: mass 0.076806 -> 0.0768058991199202
Joints:
- removed joint arm_forearm_joint
- removed joint gripper_left_pitch
- removed joint gripper_right_pitch
- removed joint pitch_yaw_joint
- removed joint roll_arm_joint
- removed joint shoulder_forearm_joint
- removed joint soulder_base_joint
- removed joint yaw_roll_joint
- added joint elbow_joint: type continuous, parent forearm_link, child elbow_link, origin xyz=0 0.30821 -0.040455 rpy=1.5708 -0.74886 -1.5708, axis 0 0 1, limit effort=10.6 velocity=6.28
- added joint forearm_shoulder_joint: type continuous, parent shoulder_link, child forearm_link, origin xyz=0 0.0656 0 rpy=0.93003 1.5708 -0.7, axis 1 0 0, limit effort=21.2 velocity=6.28
- added joint gripper_joint: type fixed, parent roll_2_link, child gripper_link, origin xyz=-0.021958 0.00027834 0.10168 rpy=3.1416 0 -0.012731, axis 0 0 0
- added joint left_finger_joint: type continuous, parent gripper_link, child left_finger_link, origin xyz=-0.038057 0 -0.0015128 rpy=2.7793 0 1.5708, axis 1 0 0, limit effort=3.2 velocity=6.28
- added joint right_finger_joint: type continuous, parent gripper_link, child right_finger_link, origin xyz=0.081977 0 -0.0015128 rpy=-3.1378 0 -1.5708, axis -1 0 0, limit effort=3.2 velocity=6.28
- added joint roll_2_joint: type continuous, parent yaw_link, child roll_2_link, origin xyz=0 -0.054822 -0.00015038 rpy=1.3649 1.5708 -0.2119, axis 0 0 1, limit effort=6.4 velocity=6.28
- added joint roll_joint: type continuous, parent elbow_link, child roll_link, origin xyz=0 0 0 rpy=1.5708 0.012731 3.1416, axis 0 0 1, limit effort=6.4 velocity=6.28
- added joint shoulder_joint: type continuous, parent arm_base_link, child shoulder_link, origin xyz=0.018961 0 0.049 rpy=1.5708 0 0, axis 0 1 0, limit effort=10.6 velocity=6.28
- added joint yaw_joint: type continuous, parent roll_link, child yaw_link, origin xyz=0 0 -0.166 rpy=1.5708 0 1.5708, axis 0 0 1, limit effort=6.4 velocity=6.28

File: doris_description/urdf/doris_description.urdf.xacro (robot description, xacro)
@@ -1,6 +1,7 @@
 <?xml version="1.0"?>
 <robot xmlns:xacro="http://www.ros.org/wiki/xacro" name="doris">
-    <xacro:include filename="$(find patrolbot_description)/urdf/patrolbot.xacro" />
+    <xacro:include filename="$(find patrolbot_description)/urdf/patrolbot_description.urdf" />
     <xacro:include filename="$(find doris_arm_description)/urdf/doris_arm_description.urdf" />
+    <xacro:include filename="$(find doris_arm_description)/urdf/hand.xacro" />
     <xacro:include filename="$(find doris_dorso_description)/urdf/doris_dorso_description.urdf" />
     <!--xacro:include filename="$(find kinect2_description)/urdf/kinect2_description.urdf.xacro" /-->
@@ -8,17 +9,62 @@
     <xacro:include filename="$(find hector_sensors_description)/urdf/hokuyo_utm30lx.urdf.xacro" />
     <xacro:include filename="$(find hector_sensors_description)/urdf/kinect_camera.urdf.xacro" />
+    <xacro:include filename="$(find lms1xx)/urdf/sick_lms1xx.urdf.xacro" />
+    <link name="base_footprint"></link>
+    <joint name="base_joint" type="fixed">
+        <child link="base_link" />
+        <parent link="base_footprint" />
+    </joint>
+    <link name="frontal_caster_link">
+        <inertial>
+            <origin xyz="0 0 0" rpy="0 0 0" />
+            <mass value="0.1" />
+            <inertia ixx="0.001" ixy="0" ixz="0" iyy="0.001" iyz="0" izz="0.001" />
+        </inertial>
+        <collision>
+            <origin xyz="0 0 0" rpy="0 0 0" />
+            <geometry>
+                <sphere radius="0.05"/>
+            </geometry>
+        </collision>
+    </link>
+    <joint name="frontal_caster_joint" type="fixed">
+        <parent link="base_link" />
+        <child link="frontal_caster_link" />
+        <origin xyz="0.2 0 0" rpy="0 0 0" />
+    </joint>
+    <link name="rear_caster_link">
+        <inertial>
+            <origin xyz="0 0 0" rpy="0 0 0" />
+            <mass value="0.1" />
+            <inertia ixx="0.001" ixy="0" ixz="0" iyy="0.001" iyz="0" izz="0.001" />
+        </inertial>
+        <collision>
+            <origin xyz="0 0 0" rpy="0 0 0" />
+            <geometry>
+                <sphere radius="0.05"/>
+            </geometry>
+        </collision>
+    </link>
+    <joint name="rear_caster_joint" type="fixed">
+        <parent link="base_link" />
+        <child link="rear_caster_link" />
+        <origin xyz="-0.2 0 0" rpy="0 0 0" />
+    </joint>
+    <!--
+    <xacro:hand ns="doris" rpy="0 0 1.570" xyz="0 0 0.1" connected_to="roll_2_link" safety_distance="0.00" use_cylinder_collision_model="false" />
+    -->
     <joint name="base_link_dorso" type="fixed">
         <parent link="base_link" />
         <child link="dorso_link" />
-        <origin xyz="-0.05 -0.01 ${base_height+0.9}" rpy="${3.1416/2} 0 3.1416" />
+        <origin xyz="0 0 0.32" rpy="0 0 0" />
     </joint>
     <joint name="dorso_arm_base" type="fixed">
         <parent link="dorso_link" />
         <child link="arm_base_link" />
-        <origin xyz="-0.28 -0.4 0.08" rpy="${3.1416/2} 0 3.1416" />
+        <origin xyz="0.2 0 0.6" rpy="0 0 0" />
     </joint>
     <xacro:sick_lms1xx />
     <joint name="laser_joint" type="fixed">
-        <origin xyz="-0.28 -0.9 0.01" rpy="${3.1416/2} 0 3.1416" />
+        <origin xyz="0.222 0 0.16" rpy="0 0 0" />
         <parent link="dorso_link" />
         <child link="laser" />
@@ -31,10 +77,10 @@
     <!--xacro:sensor_kinect prefix="" name="kinect" parent="dorso_link" cam_px="-0.18" cam_py="0" cam_pz="0.01" cam_or="${-3.1416/2}" cam_op="0" cam_oy="${3.1416/2}"></xacro:sensor_kinect-->
     <xacro:kinect_camera name="kinect2" parent="dorso_link">
-        <origin xyz="-0.25 0.025 0.01" rpy="${-3.1416/2} 3.1416 0" />
+        <origin xyz="0.2 0 1.08" rpy="0 0 0" />
     </xacro:kinect_camera>
     <joint name="dorso_head" type="fixed">
         <parent link="dorso_link" />
         <child link="head_link" />
-        <origin xyz="-0.05 0.15 0.01" rpy="${3.1416/2} 0 3.1416" />
+        <origin xyz="0 0 1.16" rpy="0 0 0" />
     </joint>
     <!--joint name="dorso_hokuyo" type="fixed">
@@ -43,6 +89,270 @@
         <origin xyz="-0.25 -0.7 0.01" rpy="${3.1416/2} ${-3.1416/2} 3.1416" />
     </joint-->
-    <xacro:hokuyo_utm30lx name="hokuyo" parent="dorso_link" ros_topic="hokuyo/scan" update_rate="30" ray_count="500" min_angle="0" max_angle="-180">
-        <origin xyz="-0.25 -0.7 0.01" rpy="${3.1416/2} ${-3.1416/2} 3.1416" />
+    <xacro:hokuyo_utm30lx name="hokuyo" parent="base_link" ros_topic="hokuyo/scan" update_rate="30" ray_count="500" min_angle="0" max_angle="-180">
+        <origin xyz="0.35 0 0.1" rpy="0 0 0" />
     </xacro:hokuyo_utm30lx>
+    <transmission name="trans_left_wheel_joint">
+        <type>transmission_interface/SimpleTransmission</type>
+        <joint name="left_wheel_joint">
+            <hardwareInterface>hardware_interface/EffortJointInterface</hardwareInterface>
+        </joint>
+        <actuator name="left_wheel_joint_motor">
+            <hardwareInterface>hardware_interface/EffortJointInterface</hardwareInterface>
+            <mechanicalReduction>1</mechanicalReduction>
+        </actuator>
+    </transmission>
+    <transmission name="trans_right_wheel_joint">
+        <type>transmission_interface/SimpleTransmission</type>
+        <joint name="right_wheel_joint">
+            <hardwareInterface>hardware_interface/EffortJointInterface</hardwareInterface>
+        </joint>
+        <actuator name="right_wheel_joint_motor">
+            <hardwareInterface>hardware_interface/EffortJointInterface</hardwareInterface>
+            <mechanicalReduction>1</mechanicalReduction>
+        </actuator>
+    </transmission>
+    <transmission name="trans_shoulder_joint">
+        <type>transmission_interface/SimpleTransmission</type>
+        <joint name="shoulder_joint">
+            <hardwareInterface>hardware_interface/EffortJointInterface</hardwareInterface>
+        </joint>
+        <actuator name="shoulder_joint_motor">
+            <hardwareInterface>hardware_interface/EffortJointInterface</hardwareInterface>
+            <mechanicalReduction>1</mechanicalReduction>
+        </actuator>
+    </transmission>
+    <transmission name="trans_forearm_shoulder_joint">
+        <type>transmission_interface/SimpleTransmission</type>
+        <joint name="forearm_shoulder_joint">
+            <hardwareInterface>hardware_interface/EffortJointInterface</hardwareInterface>
+        </joint>
+        <actuator name="forearm_shoulder_joint_motor">
+            <hardwareInterface>hardware_interface/EffortJointInterface</hardwareInterface>
+            <mechanicalReduction>1</mechanicalReduction>
+        </actuator>
+    </transmission>
+    <transmission name="trans_elbow_joint">
+        <type>transmission_interface/SimpleTransmission</type>
+        <joint name="elbow_joint">
+            <hardwareInterface>hardware_interface/EffortJointInterface</hardwareInterface>
+        </joint>
+        <actuator name="elbow_joint_motor">
+            <hardwareInterface>hardware_interface/EffortJointInterface</hardwareInterface>
+            <mechanicalReduction>1</mechanicalReduction>
+        </actuator>
+    </transmission>
+    <transmission name="trans_roll_joint">
+        <type>transmission_interface/SimpleTransmission</type>
+        <joint name="roll_joint">
+            <hardwareInterface>hardware_interface/EffortJointInterface</hardwareInterface>
+        </joint>
+        <actuator name="roll_joint_motor">
+            <hardwareInterface>hardware_interface/EffortJointInterface</hardwareInterface>
+            <mechanicalReduction>1</mechanicalReduction>
+        </actuator>
+    </transmission>
+    <transmission name="trans_yaw_joint">
+        <type>transmission_interface/SimpleTransmission</type>
+        <joint name="yaw_joint">
+            <hardwareInterface>hardware_interface/EffortJointInterface</hardwareInterface>
+        </joint>
+        <actuator name="yaw_joint_motor">
+            <hardwareInterface>hardware_interface/EffortJointInterface</hardwareInterface>
+            <mechanicalReduction>1</mechanicalReduction>
+        </actuator>
+    </transmission>
+    <transmission name="trans_roll_2_joint">
+        <type>transmission_interface/SimpleTransmission</type>
+        <joint name="roll_2_joint">
+            <hardwareInterface>hardware_interface/EffortJointInterface</hardwareInterface>
+        </joint>
+        <actuator name="roll_2_joint_motor">
+            <hardwareInterface>hardware_interface/EffortJointInterface</hardwareInterface>
+            <mechanicalReduction>1</mechanicalReduction>
+        </actuator>
+    </transmission><!--
+    <transmission name="trans_doris_finger_joint1">
+        <type>transmission_interface/SimpleTransmission</type>
+        <joint name="doris_finger_joint1">
+            <hardwareInterface>hardware_interface/EffortJointInterface</hardwareInterface>
+        </joint>
+        <actuator name="doris_finger_joint1_motor">
+            <hardwareInterface>hardware_interface/EffortJointInterface</hardwareInterface>
+            <mechanicalReduction>1</mechanicalReduction>
+        </actuator>
+    </transmission>
+    <transmission name="trans_doris_finger_joint2">
+        <type>transmission_interface/SimpleTransmission</type>
+        <joint name="doris_finger_joint2">
+            <hardwareInterface>hardware_interface/EffortJointInterface</hardwareInterface>
+        </joint>
+        <actuator name="doris_finger_joint2_motor">
+            <hardwareInterface>hardware_interface/EffortJointInterface</hardwareInterface>
+            <mechanicalReduction>1</mechanicalReduction>
+        </actuator>
+    </transmission>-->
+    <transmission name="trans_left_finger_joint">
+        <type>transmission_interface/SimpleTransmission</type>
+        <joint name="left_finger_joint">
+            <hardwareInterface>hardware_interface/EffortJointInterface</hardwareInterface>
+        </joint>
+        <actuator name="left_finger_joint_motor">
+            <hardwareInterface>hardware_interface/EffortJointInterface</hardwareInterface>
+            <mechanicalReduction>1</mechanicalReduction>
+        </actuator>
+    </transmission>
+    <transmission name="trans_right_finger_joint">
+        <type>transmission_interface/SimpleTransmission</type>
+        <joint name="right_finger_joint">
+            <hardwareInterface>hardware_interface/EffortJointInterface</hardwareInterface>
+        </joint>
+        <actuator name="right_finger_joint_motor">
+            <hardwareInterface>hardware_interface/EffortJointInterface</hardwareInterface>
+            <mechanicalReduction>1</mechanicalReduction>
+        </actuator>
+    </transmission>
+    <gazebo>
+        <plugin name="gazebo_ros_control" filename="libgazebo_ros_control.so">
+            <robotNamespace>/</robotNamespace>
+        </plugin>
+    </gazebo>
+    <transmission name="trans_left_wheel_joint">
+        <type>transmission_interface/SimpleTransmission</type>
+        <joint name="left_wheel_joint">
+            <hardwareInterface>hardware_interface/EffortJointInterface</hardwareInterface>
+        </joint>
+        <actuator name="left_wheel_joint_motor">
+            <hardwareInterface>hardware_interface/EffortJointInterface</hardwareInterface>
+            <mechanicalReduction>1</mechanicalReduction>
+        </actuator>
+    </transmission>
+    <transmission name="trans_right_wheel_joint">
+        <type>transmission_interface/SimpleTransmission</type>
+        <joint name="right_wheel_joint">
+            <hardwareInterface>hardware_interface/EffortJointInterface</hardwareInterface>
+        </joint>
+        <actuator name="right_wheel_joint_motor">
+            <hardwareInterface>hardware_interface/EffortJointInterface</hardwareInterface>
+            <mechanicalReduction>1</mechanicalReduction>
+        </actuator>
+    </transmission>
+    <gazebo>
+        <plugin name="differential_drive_controller" filename="libgazebo_ros_diff_drive.so">
+            <!-- Plugin update rate in Hz -->
+            <updateRate>50</updateRate>
+            <!-- Name of left joint, defaults to `left_joint` -->
+            <leftJoint>left_wheel_joint</leftJoint>
+            <!-- Name of right joint, defaults to `right_joint` -->
+            <rightJoint>right_wheel_joint</rightJoint>
+            <!-- The distance from the center of one wheel to the other, in meters, defaults to 0.34 m -->
+            <wheelSeparation>0.31</wheelSeparation>
+            <!-- Diameter of the wheels, in meters, defaults to 0.15 m -->
+            <wheelDiameter>0.2</wheelDiameter>
+            <!-- Wheel acceleration, in rad/s^2, defaults to 0.0 rad/s^2 -->
+            <wheelAcceleration>1.0</wheelAcceleration>
+            <!-- Maximum torque which the wheels can produce, in Nm, defaults to 5 Nm -->
+            <wheelTorque>20</wheelTorque>
+            <!-- Topic to receive geometry_msgs/Twist message commands, defaults to `cmd_vel` -->
+            <commandTopic>cmd_vel</commandTopic>
+            <!-- Topic to publish nav_msgs/Odometry messages, defaults to `odom` -->
+            <odometryTopic>odom</odometryTopic>
+            <!-- Odometry frame, defaults to `odom` -->
+            <odometryFrame>odom</odometryFrame>
+            <!-- Robot frame to calculate odometry from, defaults to `base_footprint` -->
+            <robotBaseFrame>base_footprint</robotBaseFrame>
+            <!-- Odometry source, 0 for ENCODER, 1 for WORLD, defaults to WORLD -->
+            <odometrySource>1</odometrySource>
+            <!-- Set to true to publish transforms for the wheel links, defaults to false -->
+            <publishWheelTF>false</publishWheelTF>
+            <!-- Set to true to publish transforms for the odometry, defaults to true -->
+            <publishOdom>true</publishOdom>
+            <!-- Set to true to publish sensor_msgs/JointState on /joint_states for the wheel joints, defaults to false -->
+            <publishWheelJointState>false</publishWheelJointState>
+            <!-- Set to true to swap right and left wheels, defaults to true -->
+            <legacyMode>false</legacyMode>
+        </plugin>
+    </gazebo>
+    <material name="gray_material">
+        <color rgba="0.5 0.5 0.5 1.0" />
+    </material>
+    <material name="black_material">
+        <color rgba="0.1 0.1 0.1 1.0" />
+    </material>
+    <gazebo reference="base_link">
+        <material>Gazebo/Gray</material>
+    </gazebo>
+    <gazebo reference="left_wheel_link">
+        <material>Gazebo/DarkGray</material>
+        <mu1>0.2</mu1>
+        <mu2>0.2</mu2>
+    </gazebo>
+    <gazebo reference="right_wheel_link">
+        <material>Gazebo/DarkGray</material>
+        <mu1>0.2</mu1>
+        <mu2>0.2</mu2>
+    </gazebo>
+    <gazebo reference="frontal_caster_link">
+        <mu1>0.0001</mu1>
+        <mu2>0.0001</mu2>
+    </gazebo>
+    <gazebo reference="rear_caster_link">
+        <mu1>0.0001</mu1>
+        <mu2>0.0001</mu2>
+    </gazebo>
+    <gazebo reference="dorso_link">
+        <material>Gazebo/DarkGray</material>
+    </gazebo>
+    <gazebo reference="arm_base_link">
+        <material>Gazebo/DarkGray</material>
+    </gazebo>
+    <gazebo reference="shoulder_link">
+        <material>Gazebo/DarkGray</material>
+    </gazebo>
+    <gazebo reference="forearm_link">
+        <material>Gazebo/DarkGray</material>
+    </gazebo>
+    <gazebo reference="elbow_link">
+        <material>Gazebo/DarkGray</material>
+    </gazebo>
+    <gazebo reference="roll_link">
+        <material>Gazebo/DarkGray</material>
+    </gazebo>
+    <gazebo reference="yaw_link">
+        <material>Gazebo/DarkGray</material>
+    </gazebo>
+    <gazebo reference="roll_2_link">
+        <material>Gazebo/DarkGray</material>
+    </gazebo>
+    <gazebo reference="gripper_link">
+        <material>Gazebo/DarkGray</material>
+        <mu1>1000.0</mu1>
+        <mu2>10000.0</mu2>
+        <min_depth>0.1</min_depth>
+    </gazebo>
+    <gazebo reference="left_finger_link">
+        <material>Gazebo/Gray</material>
+        <mu1>1000.0</mu1>
+        <mu2>10000.0</mu2>
+        <min_depth>0.1</min_depth>
+    </gazebo>
+    <gazebo reference="right_finger_link">
+        <material>Gazebo/Gray</material>
+        <mu1>1000.0</mu1>
+        <mu2>10000.0</mu2>
+        <min_depth>0.1</min_depth>
+    </gazebo>
+    <!--
+    <gazebo reference="doris_hand">
+        <material>Gazebo/DarkGray</material>
+    </gazebo>
+    <gazebo reference="doris_leftfinger">
+        <material>Gazebo/Gray</material>
+        <mu1>100.0</mu1>
+        <mu2>100.0</mu2>
+    </gazebo>
+    <gazebo reference="doris_rightfinger">
+        <material>Gazebo/Gray</material>
+        <mu1>100.0</mu1>
+        <mu2>100.0</mu2>
+    </gazebo>-->
 </robot>

File: doris_dorso_description/urdf/doris_dorso_description.urdf (robot description, URDF)
Before this commit: robot doris_dorso_description, 1 links, 0 joints
Links:
- link dorso_link: mass 14.0 -> 5.8385
