Commit message: smach manipulation changes

File: doris_arm_description/urdf/doris_arm_description.urdf.xacro (robot description, xacro)
@@ -3,10 +3,11 @@
      Commit Version: 1.6.0-1-g15f4949  Build Version: 1.6.7594.29634
      For more information, please see http://wiki.ros.org/sw_urdf_exporter -->
-<robot name="doris_arm_description">
+<robot xmlns:xacro="http://www.ros.org/wiki/xacro" name="doris_arm_description">
+  <xacro:property name="reduction" value="5" />
   <link name="arm_base_link">
     <inertial>
       <origin xyz="0.0032335 -3.6289E-06 0.02346" rpy="0 0 0" />
       <mass value="0.086496" />
-      <inertia ixx="2.3059E-05" ixy="1.641E-09" ixz="-1.0628E-06" iyy="4.136E-05" iyz="-2.3103E-09" izz="3.2692E-05" />
+      <inertia ixx="0.002" ixy="0.0" ixz="0.0" iyy="0.002" iyz="0.0" izz="0.002" />
     </inertial>
     <visual>
@@ -30,5 +31,5 @@
       <origin xyz="1.80019426116503E-06 0.0469908207821207 1.02798098779305E-05" rpy="0 0 0" />
       <mass value="0.187371975468428" />
-      <inertia ixx="9.67030340377893E-05" ixy="2.4150387752157E-12" ixz="4.62672389438557E-09" iyy="6.1510621044743E-05" iyz="7.92925862950938E-12" izz="6.80166975361327E-05" />
+      <inertia ixx="0.002" ixy="0.0" ixz="0.0" iyy="0.002" iyz="0.0" izz="0.002" />
     </inertial>
     <visual>
@@ -53,5 +54,6 @@
     <child link="shoulder_link" />
     <axis xyz="0 1 0" />
-    <limit effort="10.6" velocity="6.28" />
+    <limit effort="${8.4*0.2*reduction}" velocity="${6.28/reduction}" />
+    <dynamics damping="0.5" friction="0.0"/>
   </joint>
   <link name="forearm_link">
@@ -59,5 +61,5 @@
       <origin xyz="-1.08638707938674E-05 0.145957509942709 0.00428434606455026" rpy="0 0 0" />
       <mass value="0.0731491894717436" />
-      <inertia ixx="0.00041066540204533" ixy="-8.83711845735471E-13" ixz="6.82686577821298E-14" iyy="4.65670049898224E-05" iyz="5.99306396840699E-05" izz="0.000406035632117776" />
+      <inertia ixx="0.002" ixy="0.0" ixz="0.0" iyy="0.002" iyz="0.0" izz="0.002" />
     </inertial>
     <visual>
@@ -82,5 +84,6 @@
     <child link="forearm_link" />
     <axis xyz="1 0 0" />
-    <limit effort="21.2" velocity="6.28" />
+    <limit effort="${2*8.4*0.2*reduction}" velocity="${6.28/reduction}" />
+    <dynamics damping="0.5" friction="0.0"/>
   </joint>
   <link name="elbow_link">
@@ -88,5 +91,5 @@
       <origin xyz="-3.11104449999267E-05 -0.0168263295023695 0.000457294178247414" rpy="0 0 0" />
       <mass value="0.0892046248471317" />
-      <inertia ixx="4.19114884689815E-05" ixy="7.60313851177211E-09" ixz="2.31004133361254E-09" iyy="2.38301704178671E-05" iyz="-1.0628369231195E-06" izz="3.29468296689027E-05" />
+            <inertia ixx="0.002" ixy="0.0" ixz="0.0" iyy="0.002" iyz="0.0" izz="0.002" />
     </inertial>
     <visual>
@@ -111,5 +114,6 @@
     <child link="elbow_link" />
     <axis xyz="0 0 1" />
-    <limit effort="10.6" velocity="6.28" />
+    <limit effort="${8.4*0.2*reduction}" velocity="${6.28/reduction}" />
+    <dynamics damping="0.5" friction="0.0"/>
   </joint>
   <link name="roll_link">
@@ -117,5 +121,5 @@
       <origin xyz="1.19120197594746E-08 -0.010083697233814 -0.0945595691856148" rpy="0 0 0" />
       <mass value="0.108644948048519" />
-      <inertia ixx="5.28153270287721E-05" ixy="-1.47234666202985E-09" ixz="1.52885572695569E-09" iyy="5.77906922347199E-05" iyz="-3.14860619233111E-07" izz="4.90755786683178E-05" />
+            <inertia ixx="0.002" ixy="0.0" ixz="0.0" iyy="0.002" iyz="0.0" izz="0.002" />
     </inertial>
     <visual>
@@ -140,5 +144,6 @@
     <child link="roll_link" />
     <axis xyz="0 0 1" />
-    <limit effort="6.4" velocity="6.28" />
+    <limit effort="${6.0*0.2*reduction}" velocity="${6.28/reduction}" />
+    <dynamics damping="0.5" friction="0.0"/>
   </joint>
   <link name="yaw_link">
@@ -146,5 +151,5 @@
       <origin xyz="4.05516357848967E-05 -0.0160211563366842 -0.000189877443412478" rpy="0 0 0" />
       <mass value="0.0768058991199202" />
-      <inertia ixx="3.18297346758585E-05" ixy="-1.07008585036491E-08" ixz="1.50571425102129E-09" iyy="1.87354285358259E-05" iyz="-3.14989775620194E-07" izz="2.57575103945061E-05" />
+            <inertia ixx="0.002" ixy="0.0" ixz="0.0" iyy="0.002" iyz="0.0" izz="0.002" />
     </inertial>
     <visual>
@@ -169,5 +174,6 @@
     <child link="yaw_link" />
     <axis xyz="0 0 1" />
-    <limit effort="6.4" velocity="6.28" />
+    <limit effort="${6.0*0.2*reduction}" velocity="${6.28/reduction}" />
+    <dynamics damping="0.5" friction="0.0"/>
   </joint>
   <link name="roll_2_link">
@@ -175,5 +181,5 @@
       <origin xyz="3.30999898656703E-07 -0.0146248804164249 0.0456383476057014" rpy="0 0 0" />
       <mass value="0.15161780969895" />
-      <inertia ixx="6.28798955908907E-05" ixy="-2.94885470174372E-09" ixz="3.0462710061277E-09" iyy="3.67182700275411E-05" iyz="-6.30008633893171E-07" izz="5.20407281608922E-05" />
+            <inertia ixx="0.002" ixy="0.0" ixz="0.0" iyy="0.002" iyz="0.0" izz="0.002" />
     </inertial>
     <visual>
@@ -198,5 +204,6 @@
     <child link="roll_2_link" />
     <axis xyz="0 0 1" />
-    <limit effort="6.4" velocity="6.28" />
+    <limit effort="${6.0*0.2*reduction}" velocity="${6.28/reduction}" />
+    <dynamics damping="0.5" friction="0.0"/>
   </joint>
   <link name="gripper_link">
@@ -204,5 +211,5 @@
       <origin xyz="0.0230127657229507 0.000126473527769386 0.00158449770655011" rpy="0 0 0" />
       <mass value="0.0174078384350788" />
-      <inertia ixx="2.9772593568185E-06" ixy="-9.76614241037084E-11" ixz="-1.36056666866806E-20" iyy="1.55361628780027E-05" iyz="6.90655615792231E-22" izz="1.79049683506685E-05" />
+            <inertia ixx="0.002" ixy="0.0" ixz="0.0" iyy="0.002" iyz="0.0" izz="0.002" />
     </inertial>
     <visual>
@@ -232,5 +239,5 @@
       <origin xyz="-2.5501E-07 -0.0020883 0.03999" rpy="0 0 0" />
       <mass value="0.0083226" />
-      <inertia ixx="6.7417E-06" ixy="4.9528E-11" ixz="-8.9754E-11" iyy="9.1481E-06" iyz="-1.8643E-07" izz="3.3477E-06" />
+            <inertia ixx="0.002" ixy="0.0" ixz="0.0" iyy="0.002" iyz="0.0" izz="0.002" />
     </inertial>
     <visual>
@@ -255,5 +262,6 @@
     <child link="left_finger_link" />
     <axis xyz="1 0 0" />
-    <limit effort="3.2" velocity="6.28" />
+    <limit effort="${6.0*0.2*reduction/2}" velocity="${6.28/reduction}" />
+    <dynamics damping="0.5" friction="0.0"/>
   </joint>
   <link name="right_finger_link">
@@ -261,5 +269,5 @@
       <origin xyz="-2.55484871550249E-07 0.0123652457374703 0.0380876079681996" rpy="0 0 0" />
       <mass value="0.00832263335631547" />
-      <inertia ixx="6.74172247293139E-06" ixy="1.41443390446518E-11" ixz="-1.01493727185514E-10" iyy="8.28022035597717E-06" iyz="-2.07740904577141E-06" izz="4.21561599047209E-06" />
+            <inertia ixx="0.002" ixy="0.0" ixz="0.0" iyy="0.002" iyz="0.0" izz="0.002" />
     </inertial>
     <visual>
@@ -284,5 +292,6 @@
     <child link="right_finger_link" />
     <axis xyz="-1 0 0" />
-    <limit effort="3.2" velocity="6.28" />
+    <limit effort="${6.0*0.2*reduction/2}" velocity="${6.28/reduction}" />
+    <dynamics damping="0.5" friction="0.0"/>
   </joint>
 </robot>

File: doris_description/urdf/doris_description.urdf.xacro (robot description, xacro)
@@ -2,5 +2,5 @@
 <robot xmlns:xacro="http://www.ros.org/wiki/xacro" name="doris">
     <xacro:include filename="$(find patrolbot_description)/urdf/patrolbot_description.urdf" />
-    <xacro:include filename="$(find doris_arm_description)/urdf/doris_arm_description.urdf" />
+    <xacro:include filename="$(find doris_arm_description)/urdf/doris_arm_description.urdf.xacro" />
     <xacro:include filename="$(find doris_arm_description)/urdf/hand.xacro" />
     <xacro:include filename="$(find doris_dorso_description)/urdf/doris_dorso_description.urdf" />
@@ -9,4 +9,5 @@
     <xacro:include filename="$(find hector_sensors_description)/urdf/hokuyo_utm30lx.urdf.xacro" />
     <xacro:include filename="$(find hector_sensors_description)/urdf/kinect_camera.urdf.xacro" />
+    <xacro:include filename="$(find hector_sensors_description)/urdf/realsense_d435_camera.urdf.xacro" />
     <xacro:include filename="$(find lms1xx)/urdf/sick_lms1xx.urdf.xacro" />
     <link name="base_footprint"></link>
@@ -79,4 +80,9 @@
         <origin xyz="0.2 0 1.08" rpy="0 0 0" />
     </xacro:kinect_camera>
+    <!--
+    <xacro:realsense_d435_camera_with_mount name="realsense" parent="roll_2_link">
+        <origin xyz="0 0.03 0.1" rpy="-1.570 -1.570 0" />
+    </xacro:realsense_d435_camera_with_mount>
+    -->
     <joint name="dorso_head" type="fixed">
         <parent link="dorso_link" />
@@ -119,5 +125,5 @@
         <actuator name="shoulder_joint_motor">
             <hardwareInterface>hardware_interface/EffortJointInterface</hardwareInterface>
-            <mechanicalReduction>1</mechanicalReduction>
+            <mechanicalReduction>5</mechanicalReduction>
         </actuator>
     </transmission>
@@ -129,5 +135,5 @@
         <actuator name="forearm_shoulder_joint_motor">
             <hardwareInterface>hardware_interface/EffortJointInterface</hardwareInterface>
-            <mechanicalReduction>1</mechanicalReduction>
+            <mechanicalReduction>5</mechanicalReduction>
         </actuator>
     </transmission>
@@ -139,5 +145,5 @@
         <actuator name="elbow_joint_motor">
             <hardwareInterface>hardware_interface/EffortJointInterface</hardwareInterface>
-            <mechanicalReduction>1</mechanicalReduction>
+            <mechanicalReduction>5</mechanicalReduction>
         </actuator>
     </transmission>
@@ -149,5 +155,5 @@
         <actuator name="roll_joint_motor">
             <hardwareInterface>hardware_interface/EffortJointInterface</hardwareInterface>
-            <mechanicalReduction>1</mechanicalReduction>
+            <mechanicalReduction>5</mechanicalReduction>
         </actuator>
     </transmission>
@@ -159,5 +165,5 @@
         <actuator name="yaw_joint_motor">
             <hardwareInterface>hardware_interface/EffortJointInterface</hardwareInterface>
-            <mechanicalReduction>1</mechanicalReduction>
+            <mechanicalReduction>5</mechanicalReduction>
         </actuator>
     </transmission>
@@ -169,5 +175,5 @@
         <actuator name="roll_2_joint_motor">
             <hardwareInterface>hardware_interface/EffortJointInterface</hardwareInterface>
-            <mechanicalReduction>1</mechanicalReduction>
+            <mechanicalReduction>5</mechanicalReduction>
         </actuator>
     </transmission><!--
@@ -199,5 +205,5 @@
         <actuator name="left_finger_joint_motor">
             <hardwareInterface>hardware_interface/EffortJointInterface</hardwareInterface>
-            <mechanicalReduction>1</mechanicalReduction>
+            <mechanicalReduction>5</mechanicalReduction>
         </actuator>
     </transmission>
@@ -209,5 +215,5 @@
         <actuator name="right_finger_joint_motor">
             <hardwareInterface>hardware_interface/EffortJointInterface</hardwareInterface>
-            <mechanicalReduction>1</mechanicalReduction>
+            <mechanicalReduction>5</mechanicalReduction>
         </actuator>
     </transmission>
@@ -326,19 +332,36 @@
     <gazebo reference="gripper_link">
         <material>Gazebo/DarkGray</material>
-        <mu1>1000.0</mu1>
-        <mu2>10000.0</mu2>
+        <mu1>10000.0</mu1>
+        <mu2>100000.0</mu2>
         <min_depth>0.1</min_depth>
     </gazebo>
     <gazebo reference="left_finger_link">
         <material>Gazebo/Gray</material>
-        <mu1>1000.0</mu1>
-        <mu2>10000.0</mu2>
+        <mu1>10000.0</mu1>
+        <mu2>100000.0</mu2>
         <min_depth>0.1</min_depth>
     </gazebo>
     <gazebo reference="right_finger_link">
         <material>Gazebo/Gray</material>
-        <mu1>1000.0</mu1>
-        <mu2>10000.0</mu2>
+        <mu1>10000.0</mu1>
+        <mu2>100000.0</mu2>
         <min_depth>0.1</min_depth>
+    </gazebo>
+    <gazebo>
+        <plugin name="gazebo_grasp_fix" filename="libgazebo_grasp_fix.so">
+            <arm>
+                <arm_name>arm</arm_name>
+                <palm_link>roll_2_link</palm_link>
+                <gripper_link>left_finger_link</gripper_link>
+                <gripper_link>right_finger_link</gripper_link>
+            </arm>
+            <forces_angle_tolerance>100</forces_angle_tolerance>
+            <update_rate>4</update_rate>
+            <grip_count_threshold>4</grip_count_threshold>
+            <max_grip_count>8</max_grip_count>
+            <release_tolerance>0.005</release_tolerance>
+            <disable_collisions_on_attach>false</disable_collisions_on_attach>
+            <contact_topic>__default_topic__</contact_topic>
+        </plugin>
     </gazebo>
     <!--

Commit message: update joint damping and friction values

File: doris_arm_description/urdf/doris_arm_description.urdf.xacro (robot description, xacro)
@@ -55,5 +55,5 @@
     <axis xyz="0 1 0" />
     <limit effort="${8.4*0.2*reduction}" velocity="${6.28/reduction}" />
-    <dynamics damping="0.5" friction="0.0"/>
+    <dynamics damping="0.7" friction="1.0"/>
   </joint>
   <link name="forearm_link">
@@ -85,5 +85,5 @@
     <axis xyz="1 0 0" />
     <limit effort="${2*8.4*0.2*reduction}" velocity="${6.28/reduction}" />
-    <dynamics damping="0.5" friction="0.0"/>
+    <dynamics damping="0.7" friction="1.0"/>
   </joint>
   <link name="elbow_link">
@@ -115,5 +115,5 @@
     <axis xyz="0 0 1" />
     <limit effort="${8.4*0.2*reduction}" velocity="${6.28/reduction}" />
-    <dynamics damping="0.5" friction="0.0"/>
+    <dynamics damping="0.7" friction="1.0"/>
   </joint>
   <link name="roll_link">
@@ -145,5 +145,5 @@
     <axis xyz="0 0 1" />
     <limit effort="${6.0*0.2*reduction}" velocity="${6.28/reduction}" />
-    <dynamics damping="0.5" friction="0.0"/>
+    <dynamics damping="0.7" friction="1.0"/>
   </joint>
   <link name="yaw_link">
@@ -175,5 +175,5 @@
     <axis xyz="0 0 1" />
     <limit effort="${6.0*0.2*reduction}" velocity="${6.28/reduction}" />
-    <dynamics damping="0.5" friction="0.0"/>
+    <dynamics damping="0.7" friction="1.0"/>
   </joint>
   <link name="roll_2_link">
@@ -205,5 +205,5 @@
     <axis xyz="0 0 1" />
     <limit effort="${6.0*0.2*reduction}" velocity="${6.28/reduction}" />
-    <dynamics damping="0.5" friction="0.0"/>
+    <dynamics damping="0.7" friction="1.0"/>
   </joint>
   <link name="gripper_link">
@@ -263,5 +263,5 @@
     <axis xyz="1 0 0" />
     <limit effort="${6.0*0.2*reduction/2}" velocity="${6.28/reduction}" />
-    <dynamics damping="0.5" friction="0.0"/>
+    <dynamics damping="0.7" friction="1.0"/>
   </joint>
   <link name="right_finger_link">
@@ -293,5 +293,5 @@
     <axis xyz="-1 0 0" />
     <limit effort="${6.0*0.2*reduction/2}" velocity="${6.28/reduction}" />
-    <dynamics damping="0.5" friction="0.0"/>
+    <dynamics damping="0.7" friction="1.0"/>
   </joint>
 </robot>
