Commit message: Make robot with interbotix arm work in gazebo.

File: doris_arm_description/urdf/doris_arm.urdf.xacro (robot description, xacro)
@@ -9,9 +9,80 @@
     <xacro:arg name="use_world_frame" default="false"/>
     <xacro:arg name="external_urdf_loc" default=""/>
-    <xacro:arg name="load_gazebo_configs" default="false"/>
+    <xacro:arg name="load_gazebo_configs" default="true"/>
     <xacro:property name="urdf_loc" value="$(arg external_urdf_loc)"/>
     <xacro:property name="pi_offset" value="0.00001"/>
     <xacro:if value="$(arg load_gazebo_configs)">
-        <xacro:include filename="$(find interbotix_xsarm_gazebo)/config/interbotix_texture.gazebo"/>
+        <gazebo>
+            <plugin name="gazebo_ros_control" filename="libgazebo_ros_control.so">
+            <robotSimType>gazebo_ros_control/DefaultRobotHWSim</robotSimType>
+            <legacyModeNS>true</legacyModeNS>
+            <robotNamespace>/$(arg robot_name)</robotNamespace>
+            </plugin>
+        </gazebo>
+        <gazebo reference="$(arg robot_name)/$(arg base_link_frame)">
+            <material>Gazebo/DarkGray</material>
+            <dampingFactor>0.1</dampingFactor>
+        </gazebo>
+        <gazebo reference="$(arg robot_name)/shoulder_link">
+            <material>Gazebo/DarkGray</material>
+            <dampingFactor>0.1</dampingFactor>
+        </gazebo>
+        <gazebo reference="$(arg robot_name)/upper_arm_link">
+            <material>Gazebo/DarkGray</material>
+            <dampingFactor>0.1</dampingFactor>
+        </gazebo>
+        <gazebo reference="$(arg robot_name)/forearm_link">
+            <material>Gazebo/DarkGray</material>
+            <dampingFactor>0.1</dampingFactor>
+        </gazebo>
+        <gazebo reference="$(arg robot_name)/upper_forearm_link">
+            <material>Gazebo/DarkGray</material>
+            <dampingFactor>0.1</dampingFactor>
+        </gazebo>
+        <gazebo reference="$(arg robot_name)/lower_forearm_link">
+            <material>Gazebo/DarkGray</material>
+            <dampingFactor>0.1</dampingFactor>
+        </gazebo>
+        <gazebo reference="$(arg robot_name)/wrist_link">
+            <material>Gazebo/DarkGray</material>
+            <dampingFactor>0.1</dampingFactor>
+        </gazebo>
+        <gazebo reference="$(arg robot_name)/gripper_link">
+            <material>Gazebo/DarkGray</material>
+            <dampingFactor>0.1</dampingFactor>
+        </gazebo>
+        <gazebo reference="$(arg robot_name)/gripper_prop_link">
+            <material>Gazebo/DarkGray</material>
+            <dampingFactor>0.1</dampingFactor>
+        </gazebo>
+        <gazebo reference="$(arg robot_name)/gripper_bar_link">
+            <material>Gazebo/DarkGray</material>
+        </gazebo>
+        <gazebo reference="$(arg robot_name)/left_finger_link">
+            <material>Gazebo/DarkGray</material>
+            <dampingFactor>0.1</dampingFactor>
+        </gazebo>
+        <gazebo reference="$(arg robot_name)/right_finger_link">
+            <material>Gazebo/DarkGray</material>
+            <dampingFactor>0.1</dampingFactor>
+        </gazebo>
+        <gazebo reference="$(arg robot_name)/ar_tag_link">
+            <material>Gazebo/DarkGray</material>
+        </gazebo>
+        <gazebo reference="ee_arm">
+            <disableFixedJointLumping>true</disableFixedJointLumping>
+        </gazebo>
+        <gazebo reference="ar_tag">
+            <disableFixedJointLumping>true</disableFixedJointLumping>
+        </gazebo>
+        <gazebo reference="gripper_bar">
+            <disableFixedJointLumping>true</disableFixedJointLumping>
+        </gazebo>
+        <gazebo reference="ee_bar">
+            <disableFixedJointLumping>true</disableFixedJointLumping>
+        </gazebo>
+        <gazebo reference="ee_gripper">
+            <disableFixedJointLumping>true</disableFixedJointLumping>
+        </gazebo>
     </xacro:if>
     <material name="interbotix_black">

File: doris_description/urdf/doris_no_arm.urdf.xacro (robot description, xacro)
@@ -11,5 +11,5 @@
     <xacro:include filename="$(find doris_sensors_description)/urdf/sick_lms1xx.urdf.xacro" />
     <xacro:include filename="$(find doris_sensors_description)/urdf/materials.xacro" />
-    <!--xacro:include filename="$(find doris_sensors_description)/urdf/kinect_camera.urdf.xacro" /-->
+    <xacro:include filename="$(find doris_sensors_description)/urdf/kinect_camera.urdf.xacro" />
     <xacro:include filename="$(find hector_sensors_description)/urdf/realsense_d435_camera.urdf.xacro" />
     <!--xacro:include filename="$(find lms1xx)/urdf/sick_lms1xx.urdf.xacro" /-->
@@ -80,7 +80,7 @@
     </joint-->
     <!--xacro:sensor_kinect prefix="" name="kinect" parent="dorso_link" cam_px="-0.18" cam_py="0" cam_pz="0.01" cam_or="${-3.1416/2}" cam_op="0" cam_oy="${3.1416/2}"></xacro:sensor_kinect-->
-    <!--xacro:kinect_camera name="kinect2" parent="dorso_link">
+    <xacro:kinect_camera name="kinect2" parent="dorso_link">
         <origin xyz="0.1362 0 0.8465" rpy="0 0 0" />
-    </xacro:kinect_camera-->
+    </xacro:kinect_camera>
     <!--
     <xacro:realsense_d435_camera_with_mount name="realsense" parent="roll_2_link">
@@ -139,5 +139,5 @@
             <wheelTorque>200</wheelTorque>
             <!-- Topic to receive geometry_msgs/Twist message commands, defaults to `cmd_vel` -->
-            <commandTopic>cmd_vel</commandTopic>
+            <commandTopic>RosAria/cmd_vel</commandTopic>
             <!-- Topic to publish nav_msgs/Odometry messages, defaults to `odom` -->
             <odometryTopic>odom</odometryTopic>

File: doris_sensors_description/urdf/kinect_camera.urdf.xacro (robot description, xacro)
@@ -70,9 +70,9 @@
           </camera>
           <plugin name="${name}_camera_controller" filename="libgazebo_ros_openni_kinect.so">
-            <imageTopicName>${name}/rgb/image_raw</imageTopicName>
-            <cameraInfoTopicName>${name}/rgb/camera_info</cameraInfoTopicName>
-            <depthImageTopicName>${name}/depth/image_raw</depthImageTopicName>
-            <depthImageCameraInfoTopicName>${name}/depth/camera_info</depthImageCameraInfoTopicName>
-            <pointCloudTopicName>${name}/depth/points</pointCloudTopicName>
+            <imageTopicName>butia_vision/bvb/image_rgb</imageTopicName>
+            <cameraInfoTopicName>butia_vision/bvb/camera_info</cameraInfoTopicName>
+            <depthImageTopicName>butia_vision/bvb/image_depth</depthImageTopicName>
+            <depthImageCameraInfoTopicName>butia_vision/bvb/camera_info_depth</depthImageCameraInfoTopicName>
+            <pointCloudTopicName>butia_vision/bvb/points</pointCloudTopicName>
             <frameName>${name}_depth_optical_frame</frameName>
             <robotNamespace>/</robotNamespace>
