Commit message: Fixed grammar error.

File: doris_head_description/urdf/doris_head.urdf (robot description, URDF)
Before this commit: robot doris_head, 16 links, 15 joints
Links:
- removed link rigth_eye_horizontal_link
- removed link rigth_eye_vertical_link
- removed link rigth_inferior_eyelid_link
- removed link rigth_superior_eyelid_link
- added link right_eye_horizontal_link, mass 0.001
- added link right_eye_vertical_link, mass 0.001; visual mesh filename=package://rosto_teste/meshes/dae/Cube.007.dae scale=0.001 0.001 0.001
- added link right_inferior_eyelid_link, mass 0.001; visual mesh filename=package://rosto_teste/meshes/dae/Plane.013.dae scale=0.001 0.001 0.001
- added link right_superior_eyelid_link, mass 0.001; visual mesh filename=package://rosto_teste/meshes/dae/Plane.014.dae scale=0.001 0.001 0.001
Joints:
- removed joint rigth_eye_horizontal_joint
- removed joint rigth_eye_vertical_joint
- removed joint rigth_inferior_eyelid_joint
- removed joint rigth_superior_eyelid_joint
- added joint right_eye_horizontal_joint: type revolute, parent head_link, child right_eye_horizontal_link, origin xyz=0.09352 -0.08739 0.01605 rpy=1.5708 0 0, axis 0 0 1.0, limit lower=-0.27453 upper=0.4 effort=6.5 velocity=1000
- added joint right_eye_vertical_joint: type revolute, parent right_eye_horizontal_link, child right_eye_vertical_link, origin xyz=0 0 0 rpy=1.5708 0 0, axis 0 0 1.0, limit lower=-0.2 upper=0.7854 effort=6.5 velocity=1000
- added joint right_inferior_eyelid_joint: type revolute, parent head_link, child right_inferior_eyelid_link, origin xyz=0.09188 -0.08649 -0.00398 rpy=-3.14159 0 0, axis 0 0 1.0, limit lower=-0.17 upper=0.7854 effort=6.5 velocity=1000
- added joint right_superior_eyelid_joint: type revolute, parent head_link, child right_superior_eyelid_link, origin xyz=0.09073 -0.08626 0.03037 rpy=0 0 0, axis 0 0 1.0, limit lower=-0.4 upper=0.17 effort=6.5 velocity=1000

Commit message: Changed head controllers.

File: doris_head_description/urdf/doris_head.urdf (robot description, URDF)
Before this commit: robot doris_head, 16 links, 15 joints
Joints:
- joint horizontal_neck_joint: limit lower=-0.86 upper=0.86 effort=6.5 velocity=1000 -> lower=-0.86 upper=0.86 effort=1.0 velocity=10
- joint jaw_joint: limit lower=0 upper=0.5 effort=6.5 velocity=1000 -> lower=0 upper=0.5 effort=1.0 velocity=10
- joint left_eye_horizontal_joint: limit lower=-0.27453 upper=0.7854 effort=6.5 velocity=1000 -> lower=-0.27453 upper=0.7854 effort=1.0 velocity=10
- joint left_eye_vertical_joint: limit lower=-0.17453 upper=0.7854 effort=6.5 velocity=1000 -> lower=-0.17453 upper=0.7854 effort=1.0 velocity=10
- joint left_inferior_eyelid_joint: limit lower=-0.17453 upper=0.7854 effort=6.5 velocity=1000 -> lower=-0.17453 upper=0.7854 effort=1.0 velocity=10
- joint left_rotacional_eyebrow_joint: limit lower=-0.17453 upper=0.4 effort=6.5 velocity=1000 -> lower=-0.17453 upper=0.4 effort=1.0 velocity=10
- joint left_superior_eyelid_joint: limit lower=-0.17453 upper=0.4 effort=6.5 velocity=1000 -> lower=-0.17453 upper=0.4 effort=1.0 velocity=10
- joint left_vertical_eyebrow_joint: limit lower=0 upper=0.02 effort=6.5 velocity=1000 -> lower=0 upper=0.02 effort=1.0 velocity=10
- joint right_eye_horizontal_joint: limit lower=-0.27453 upper=0.4 effort=6.5 velocity=1000 -> lower=-0.27453 upper=0.4 effort=1.0 velocity=10
- joint right_eye_vertical_joint: limit lower=-0.2 upper=0.7854 effort=6.5 velocity=1000 -> lower=-0.2 upper=0.7854 effort=1.0 velocity=10
- joint right_inferior_eyelid_joint: limit lower=-0.17 upper=0.7854 effort=6.5 velocity=1000 -> lower=-0.17 upper=0.7854 effort=1.0 velocity=10
- joint right_rotacional_eyebrow_joint: limit lower=-0.4 upper=0.17453 effort=6.5 velocity=1000 -> lower=-0.4 upper=0.17453 effort=1.0 velocity=10
- joint right_superior_eyelid_joint: limit lower=-0.4 upper=0.17 effort=6.5 velocity=1000 -> lower=-0.4 upper=0.17 effort=1.0 velocity=10
- joint right_vertical_eyebrow_joint: limit lower=0 upper=0.02 effort=6.5 velocity=1000 -> lower=0 upper=0.02 effort=1.0 velocity=10
- joint vertical_neck_joint: limit lower=0 upper=0.5 effort=6.5 velocity=1000 -> lower=0 upper=0.5 effort=1.0 velocity=10

Commit message: some modifications

File: doris_head_description/urdf/doris_head.urdf (robot description, URDF)
Before this commit: robot doris_head, 16 links, 15 joints
Links:
- link head_link: geometry visual mesh filename=package://doris_head_description/meshes/dae/Cube.001.dae scale=0.001 0.001 0.001
- link jaw_link: geometry visual mesh filename=package://doris_head_description/meshes/dae/Plane.012.dae scale=0.001 0.001 0.001
- link left_eye_vertical_link: geometry visual mesh filename=package://doris_head_description/meshes/dae/Cube.002.dae scale=0.001 0.001 0.001
- link left_inferior_eyelid_link: geometry visual mesh filename=package://doris_head_description/meshes/dae/Plane.015.dae scale=0.001 0.001 0.001
- link left_rotacional_eyebrow_link: geometry visual mesh filename=package://doris_head_description/meshes/dae/Cylinder.004.dae scale=0.001 0.001 0.001
- link left_superior_eyelid_link: geometry visual mesh filename=package://doris_head_description/meshes/dae/Plane.001.dae scale=0.001 0.001 0.001
- link neck_link: geometry visual mesh filename=package://doris_head_description/meshes/dae/Cube.055.dae scale=0.01 0.01 0.01
- link right_eye_vertical_link: geometry visual mesh filename=package://doris_head_description/meshes/dae/Cube.007.dae scale=0.001 0.001 0.001
- link right_inferior_eyelid_link: geometry visual mesh filename=package://doris_head_description/meshes/dae/Plane.013.dae scale=0.001 0.001 0.001
- link right_rotacional_eyebrow_link: geometry visual mesh filename=package://doris_head_description/meshes/dae/Cylinder.005.dae scale=0.001 0.001 0.001
- link right_superior_eyelid_link: geometry visual mesh filename=package://doris_head_description/meshes/dae/Plane.014.dae scale=0.001 0.001 0.001
