Commit message: fixed some bugs

File: doris_description/urdf/doris_description.urdf.xacro (robot description, xacro)
@@ -30,6 +30,6 @@
     </joint-->
     <!--xacro:sensor_kinect prefix="" name="kinect" parent="dorso_link" cam_px="-0.18" cam_py="0" cam_pz="0.01" cam_or="${-3.1416/2}" cam_op="0" cam_oy="${3.1416/2}"></xacro:sensor_kinect-->
-    <xacro:kinect_camera name="kinect" parent="dorso_link">
-        <origin xyz="-0.2 0.025 0.01" rpy="${-3.1416/2} 3.1416 0" />
+    <xacro:kinect_camera name="kinect2" parent="dorso_link">
+        <origin xyz="-0.25 0.025 0.01" rpy="${-3.1416/2} 3.1416 0" />
     </xacro:kinect_camera>
     <joint name="dorso_head" type="fixed">
@@ -43,5 +43,5 @@
         <origin xyz="-0.25 -0.7 0.01" rpy="${3.1416/2} ${-3.1416/2} 3.1416" />
     </joint-->
-    <xacro:hokuyo_utm30lx name="hokuyo" parent="dorso_link" ros_topic="hokuyo/scan" update_rate="40" ray_count="1000" min_angle="0" max_angle="-180">
+    <xacro:hokuyo_utm30lx name="hokuyo" parent="dorso_link" ros_topic="hokuyo/scan" update_rate="30" ray_count="500" min_angle="0" max_angle="-180">
         <origin xyz="-0.25 -0.7 0.01" rpy="${3.1416/2} ${-3.1416/2} 3.1416" />
     </xacro:hokuyo_utm30lx>

File: patrolbot_description/urdf/caster.xacro (robot description, xacro)
@@ -29,6 +29,6 @@
         </joint>
         <gazebo reference="${prefix}_caster_wheel">
-            <mu1 value="0.0001" />
-            <mu2 value="0.0001" />
+            <mu1 value="0.0000001" />
+            <mu2 value="0.0000001" />
             <kp value="10000000.0" />
             <kd value="1.0" />

File: patrolbot_description/urdf/patrolbot.xacro (robot description, xacro)
@@ -73,5 +73,5 @@
             <wheelAcceleration>0.0</wheelAcceleration>
             <!-- Maximum torque which the wheels can produce, in Nm, defaults to 5 Nm -->
-            <wheelTorque>120</wheelTorque>
+            <wheelTorque>240</wheelTorque>
             <!-- Topic to receive geometry_msgs/Twist message commands, defaults to `cmd_vel` -->
             <commandTopic>cmd_vel</commandTopic>

Commit message: fixing hokuyo topic and position

File: doris_description/urdf/doris_description.urdf.xacro (robot description, xacro)
@@ -95,6 +95,6 @@
         <origin xyz="-0.25 -0.7 0.01" rpy="${3.1416/2} ${-3.1416/2} 3.1416" />
     </joint-->
-    <xacro:hokuyo_utm30lx name="hokuyo" parent="base_link" ros_topic="hokuyo/scan" update_rate="30" ray_count="500" min_angle="0" max_angle="-180">
-        <origin xyz="0.35 0 0.1" rpy="0 0 0" />
+    <xacro:hokuyo_utm30lx name="hokuyo" parent="base_link" ros_topic="scan2" update_rate="30" ray_count="500" min_angle="0" max_angle="-180">
+        <origin xyz="0.35 0 0.01" rpy="3.14 0 0" />
     </xacro:hokuyo_utm30lx>
     <transmission name="trans_left_wheel_joint">

Commit message: adjusting arm and kinect position to better see and manipulate go and get it objects

File: doris_description/urdf/doris_description.urdf.xacro (robot description, xacro)
@@ -63,5 +63,5 @@
         <parent link="dorso_link" />
         <child link="arm_base_link" />
-        <origin xyz="0.2 0 0.6" rpy="0 0 0" />
+        <origin xyz="0.2 0 0.4" rpy="0 0 0" />
     </joint>
     <xacro:sick_lms1xx />
@@ -78,5 +78,5 @@
     <!--xacro:sensor_kinect prefix="" name="kinect" parent="dorso_link" cam_px="-0.18" cam_py="0" cam_pz="0.01" cam_or="${-3.1416/2}" cam_op="0" cam_oy="${3.1416/2}"></xacro:sensor_kinect-->
     <xacro:kinect_camera name="kinect2" parent="dorso_link">
-        <origin xyz="0.2 0 1.08" rpy="0 0 0" />
+        <origin xyz="0.23 0 0.9" rpy="0 0.348 0" />
     </xacro:kinect_camera>
     <!--

Commit message: lowering hokuyo to detect very small objects

File: doris_description/urdf/doris_description.urdf.xacro (robot description, xacro)
@@ -96,5 +96,5 @@
     </joint-->
     <xacro:hokuyo_utm30lx name="hokuyo" parent="base_link" ros_topic="scan2" update_rate="30" ray_count="500" min_angle="0" max_angle="-180">
-        <origin xyz="0.35 0 0.01" rpy="3.14 0 0" />
+        <origin xyz="0.35 0 -0.01" rpy="3.14 0 0" />
     </xacro:hokuyo_utm30lx>
     <transmission name="trans_left_wheel_joint">

Commit message: URDF doris_head.

File: doris_description/urdf/doris_description.urdf.xacro (robot description, xacro)
@@ -87,5 +87,5 @@
     <joint name="dorso_head" type="fixed">
         <parent link="dorso_link" />
-        <child link="head_link" />
+        <child link="head_root" />
         <origin xyz="0 0 1.16" rpy="0 0 0" />
     </joint>

File: doris_head_description/urdf/doris_head.urdf (robot description, URDF)
Before this commit: robot doris_head, 1 links, 0 joints
Links:
- added link head_root, mass 0.001
- added link jaw_link, mass 0.001; visual mesh filename=package://rosto_teste/meshes/dae/Plane.012.dae scale=0.001 0.001 0.001
- added link left_eye_horizontal_link, mass 0.001
- added link left_eye_vertical_link, mass 0.001; visual mesh filename=package://rosto_teste/meshes/dae/Cube.002.dae scale=0.001 0.001 0.001
- added link left_inferior_eyelid_link, mass 0.001; visual mesh filename=package://rosto_teste/meshes/dae/Plane.015.dae scale=0.001 0.001 0.001
- added link left_rotacional_eyebrow_link, mass 0.001; visual mesh filename=package://rosto_teste/meshes/dae/Cylinder.004.dae scale=0.001 0.001 0.001
- added link left_superior_eyelid_link, mass 0.001; visual mesh filename=package://rosto_teste/meshes/dae/Plane.001.dae scale=0.001 0.001 0.001
- added link left_vertical_eyebrow_link, mass 0.001
- added link neck_link, mass 0.001; visual mesh filename=package://rosto_teste/meshes/dae/Cube.055.dae scale=0.01 0.01 0.01
- added link right_rotacional_eyebrow_link, mass 0.001; visual mesh filename=package://rosto_teste/meshes/dae/Cylinder.005.dae scale=0.001 0.001 0.001
- added link right_vertical_eyebrow_link, mass 0.001
- added link rigth_eye_horizontal_link, mass 0.001
- added link rigth_eye_vertical_link, mass 0.001; visual mesh filename=package://rosto_teste/meshes/dae/Cube.007.dae scale=0.001 0.001 0.001
- added link rigth_inferior_eyelid_link, mass 0.001; visual mesh filename=package://rosto_teste/meshes/dae/Plane.013.dae scale=0.001 0.001 0.001
- added link rigth_superior_eyelid_link, mass 0.001; visual mesh filename=package://rosto_teste/meshes/dae/Plane.014.dae scale=0.001 0.001 0.001
- link head_link: mass 0.2 -> 0.001; geometry visual mesh filename=package://rosto_teste/meshes/dae/Cube.001.dae scale=0.001 0.001 0.001
Joints:
- added joint horizontal_neck_joint: type revolute, parent head_root, child neck_link, origin xyz=0 0 0 rpy=0 0 1.5708, axis 0 0 1.0, limit lower=-0.86 upper=0.86 effort=6.5 velocity=1000
- added joint jaw_joint: type revolute, parent head_link, child jaw_link, origin xyz=0.00668 -0.10888 0.05845 rpy=0 0 0, axis 0 0 1.0, limit lower=0 upper=0.5 effort=6.5 velocity=1000
- added joint left_eye_horizontal_joint: type revolute, parent head_link, child left_eye_horizontal_link, origin xyz=0.09352 -0.08739 -0.05892 rpy=1.5708 0 0, axis 0 0 1.0, limit lower=-0.27453 upper=0.7854 effort=6.5 velocity=1000
- added joint left_eye_vertical_joint: type revolute, parent left_eye_horizontal_link, child left_eye_vertical_link, origin xyz=0 0 0 rpy=1.5708 0 0, axis 0 0 1.0, limit lower=-0.17453 upper=0.7854 effort=6.5 velocity=1000
- added joint left_inferior_eyelid_joint: type revolute, parent head_link, child left_inferior_eyelid_link, origin xyz=0.09208 -0.08718 -0.0824 rpy=-3.14159 -0.06113 0, axis 0 0 1.0, limit lower=-0.17453 upper=0.7854 effort=6.5 velocity=1000
- added joint left_rotacional_eyebrow_joint: type revolute, parent left_vertical_eyebrow_link, child left_rotacional_eyebrow_link, origin xyz=0 0 0 rpy=2e-05 1.57091 6e-05, axis 0 0 1.0, limit lower=-0.17453 upper=0.4 effort=6.5 velocity=1000
- added joint left_superior_eyelid_joint: type revolute, parent head_link, child left_superior_eyelid_link, origin xyz=0.09123 -0.0871 -0.04284 rpy=0 0.06113 0, axis 0 0 1.0, limit lower=-0.17453 upper=0.4 effort=6.5 velocity=1000
- added joint left_vertical_eyebrow_joint: type prismatic, parent head_link, child left_vertical_eyebrow_link, origin xyz=0.1119 -0.12427 -0.0587 rpy=1.5708 0 -0.00012, axis 0 0 1.0, limit lower=0 upper=0.02 effort=6.5 velocity=1000
- added joint right_rotacional_eyebrow_joint: type revolute, parent right_vertical_eyebrow_link, child right_rotacional_eyebrow_link, origin xyz=0 0 0 rpy=0 1.5708 0, axis 0 0 1.0, limit lower=-0.4 upper=0.17453 effort=6.5 velocity=1000
- added joint right_vertical_eyebrow_joint: type prismatic, parent head_link, child right_vertical_eyebrow_link, origin xyz=0.1119 -0.12289 0.01565 rpy=1.5708 0 0, axis 0 0 1.0, limit lower=0 upper=0.02 effort=6.5 velocity=1000
- added joint rigth_eye_horizontal_joint: type revolute, parent head_link, child rigth_eye_horizontal_link, origin xyz=0.09352 -0.08739 0.01605 rpy=1.5708 0 0, axis 0 0 1.0, limit lower=-0.27453 upper=0.4 effort=6.5 velocity=1000
- added joint rigth_eye_vertical_joint: type revolute, parent rigth_eye_horizontal_link, child rigth_eye_vertical_link, origin xyz=0 0 0 rpy=1.5708 0 0, axis 0 0 1.0, limit lower=-0.2 upper=0.7854 effort=6.5 velocity=1000
- added joint rigth_inferior_eyelid_joint: type revolute, parent head_link, child rigth_inferior_eyelid_link, origin xyz=0.09188 -0.08649 -0.00398 rpy=-3.14159 0 0, axis 0 0 1.0, limit lower=-0.17 upper=0.7854 effort=6.5 velocity=1000
- added joint rigth_superior_eyelid_joint: type revolute, parent head_link, child rigth_superior_eyelid_link, origin xyz=0.09073 -0.08626 0.03037 rpy=0 0 0, axis 0 0 1.0, limit lower=-0.4 upper=0.17 effort=6.5 velocity=1000
- added joint vertical_neck_joint: type revolute, parent neck_link, child head_link, origin xyz=0.02367 -0.00121 0.01929 rpy=-1.5708 0 -1.5708, axis 0 0 1.0, limit lower=0 upper=0.5 effort=6.5 velocity=1000

Commit message: rail construction

File: doris_description/urdf/doris_description.urdf.xacro (robot description, xacro)
@@ -60,8 +60,11 @@
         <origin xyz="0 0 0.32" rpy="0 0 0" />
     </joint>
-    <joint name="dorso_arm_base" type="fixed">
+    <joint name="dorso_arm_base" type="prismatic">
         <parent link="dorso_link" />
         <child link="arm_base_link" />
         <origin xyz="0.2 0 0.4" rpy="0 0 0" />
+        <axis xyz="0 0 1"/>
+        <dynamics damping="0.7" friction="1.0"/>
+        <limit effort="100000.0" lower="-0.2" upper="0.5" velocity="0.5"/>
     </joint>
     <xacro:sick_lms1xx />
@@ -104,4 +107,14 @@
         </joint>
         <actuator name="left_wheel_joint_motor">
+            <hardwareInterface>hardware_interface/EffortJointInterface</hardwareInterface>
+            <mechanicalReduction>1</mechanicalReduction>
+        </actuator>
+    </transmission>
+    <transmission name="trans_dorso_arm_base_joint">
+        <type>transmission_interface/SimpleTransmission</type>
+        <joint name="dorso_arm_base">
+            <hardwareInterface>hardware_interface/EffortJointInterface</hardwareInterface>
+        </joint>
+        <actuator name="dorso_arm_linear_actuator">
             <hardwareInterface>hardware_interface/EffortJointInterface</hardwareInterface>
             <mechanicalReduction>1</mechanicalReduction>

Commit message: fixing patrol and hokuyo

File: doris_description/urdf/doris_description.urdf.xacro (robot description, xacro)
@@ -58,17 +58,17 @@
         <parent link="base_link" />
         <child link="dorso_link" />
-        <origin xyz="0 0 0.32" rpy="0 0 0" />
+        <origin xyz="0 0 0.28" rpy="0 0 0" />
     </joint>
     <joint name="dorso_arm_base" type="prismatic">
         <parent link="dorso_link" />
         <child link="arm_base_link" />
-        <origin xyz="0.2 0 0.4" rpy="0 0 0" />
+        <origin xyz="0.20 0 0" rpy="0 0 0" />
         <axis xyz="0 0 1"/>
         <dynamics damping="0.7" friction="1.0"/>
-        <limit effort="100000.0" lower="-0.2" upper="0.5" velocity="0.5"/>
+        <limit effort="10000.0" lower="0" upper="0.5" velocity="0.5"/>
     </joint>
     <xacro:sick_lms1xx />
     <joint name="laser_joint" type="fixed">
-        <origin xyz="0.222 0 0.16" rpy="0 0 0" />
+        <origin xyz="0.222 0 -0.07" rpy="0 0 0" />
         <parent link="dorso_link" />
         <child link="laser" />
@@ -99,5 +99,5 @@
     </joint-->
     <xacro:hokuyo_utm30lx name="hokuyo" parent="base_link" ros_topic="scan2" update_rate="30" ray_count="500" min_angle="0" max_angle="-180">
-        <origin xyz="0.35 0 -0.01" rpy="3.14 0 0" />
+        <origin xyz="0.32 0 0" rpy="3.14 0 0" />
     </xacro:hokuyo_utm30lx>
     <transmission name="trans_left_wheel_joint">

File: patrolbot_description/urdf/patrolbot.xacro (robot description, xacro)
@@ -27,5 +27,5 @@
             <origin xyz="0 0 0" rpy="0 0 0" />
             <geometry>
-                <mesh filename="package://patrolbot_description/meshes/hull.stl" />
+                <mesh filename="package://patrolbot_description/meshes/hull.stl" scale = "1 1 0.7"/>
             </geometry>
         </collision>
@@ -33,5 +33,5 @@
             <origin xyz="0 0 0" rpy="0 0 0" />
             <geometry>
-                <mesh filename="package://patrolbot_description/meshes/hull.stl" />
+                <mesh filename="package://patrolbot_description/meshes/hull.stl" scale = "1 1 0.7"/>
             </geometry>
         </visual>

File: patrolbot_description/urdf/patrolbot_description.urdf (robot description, URDF)
Before this commit: robot patrolbot_description, 3 links, 2 joints
Links:
- link base_link: geometry collision mesh filename=package://patrolbot_description/meshes/hull.stl scale=1 1 0.8; visual mesh filename=package://patrolbot_description/meshes/hull.stl scale=1 1 0.8
- link left_wheel_link: geometry collision mesh filename=package://patrolbot_description/meshes/left_wheel_link.STL; visual mesh filename=package://patrolbot_description/meshes/left_wheel.stl
- link right_wheel_link: geometry collision mesh filename=package://patrolbot_description/meshes/right_wheel_link.STL; visual mesh filename=package://patrolbot_description/meshes/right_wheel.stl

Commit message: increasing damping and friction in dorso_arm_base joint

File: doris_description/urdf/doris_description.urdf.xacro (robot description, xacro)
@@ -65,6 +65,6 @@
         <origin xyz="0.20 0 0" rpy="0 0 0" />
         <axis xyz="0 0 1"/>
-        <dynamics damping="0.7" friction="1.0"/>
-        <limit effort="10000.0" lower="0" upper="0.5" velocity="0.5"/>
+        <limit effort="2000.0" lower="0.02" upper="0.5" velocity="0.5"/>
+        <dynamics damping="20" friction="5"/>
     </joint>
     <xacro:sick_lms1xx />

Commit message: working on ground pickup

File: doris_description/urdf/doris_description.urdf.xacro (robot description, xacro)
@@ -66,5 +66,5 @@
         <axis xyz="0 0 1"/>
         <limit effort="2000.0" lower="0.02" upper="0.5" velocity="0.5"/>
-        <dynamics damping="20" friction="5"/>
+        <dynamics damping="0.5" friction="0.1"/>
     </joint>
     <xacro:sick_lms1xx />
@@ -81,5 +81,5 @@
     <!--xacro:sensor_kinect prefix="" name="kinect" parent="dorso_link" cam_px="-0.18" cam_py="0" cam_pz="0.01" cam_or="${-3.1416/2}" cam_op="0" cam_oy="${3.1416/2}"></xacro:sensor_kinect-->
     <xacro:kinect_camera name="kinect2" parent="dorso_link">
-        <origin xyz="0.23 0 0.9" rpy="0 0.348 0" />
+        <origin xyz="0.23 0 0.82" rpy="0 0.348 0" />
     </xacro:kinect_camera>
     <!--
@@ -114,8 +114,8 @@
         <type>transmission_interface/SimpleTransmission</type>
         <joint name="dorso_arm_base">
-            <hardwareInterface>hardware_interface/EffortJointInterface</hardwareInterface>
+            <hardwareInterface>hardware_interface/PositionJointInterface</hardwareInterface>
         </joint>
         <actuator name="dorso_arm_linear_actuator">
-            <hardwareInterface>hardware_interface/EffortJointInterface</hardwareInterface>
+            <hardwareInterface>hardware_interface/PositionJointInterface</hardwareInterface>
             <mechanicalReduction>1</mechanicalReduction>
         </actuator>
@@ -134,8 +134,8 @@
         <type>transmission_interface/SimpleTransmission</type>
         <joint name="shoulder_joint">
-            <hardwareInterface>hardware_interface/EffortJointInterface</hardwareInterface>
+            <hardwareInterface>hardware_interface/PositionJointInterface</hardwareInterface>
         </joint>
         <actuator name="shoulder_joint_motor">
-            <hardwareInterface>hardware_interface/EffortJointInterface</hardwareInterface>
+            <hardwareInterface>hardware_interface/PositionJointInterface</hardwareInterface>
             <mechanicalReduction>5</mechanicalReduction>
         </actuator>
@@ -144,8 +144,8 @@
         <type>transmission_interface/SimpleTransmission</type>
         <joint name="forearm_shoulder_joint">
-            <hardwareInterface>hardware_interface/EffortJointInterface</hardwareInterface>
+            <hardwareInterface>hardware_interface/PositionJointInterface</hardwareInterface>
         </joint>
         <actuator name="forearm_shoulder_joint_motor">
-            <hardwareInterface>hardware_interface/EffortJointInterface</hardwareInterface>
+            <hardwareInterface>hardware_interface/PositionJointInterface</hardwareInterface>
             <mechanicalReduction>5</mechanicalReduction>
         </actuator>
@@ -154,8 +154,8 @@
         <type>transmission_interface/SimpleTransmission</type>
         <joint name="elbow_joint">
-            <hardwareInterface>hardware_interface/EffortJointInterface</hardwareInterface>
+            <hardwareInterface>hardware_interface/PositionJointInterface</hardwareInterface>
         </joint>
         <actuator name="elbow_joint_motor">
-            <hardwareInterface>hardware_interface/EffortJointInterface</hardwareInterface>
+            <hardwareInterface>hardware_interface/PositionJointInterface</hardwareInterface>
             <mechanicalReduction>5</mechanicalReduction>
         </actuator>
@@ -164,8 +164,8 @@
         <type>transmission_interface/SimpleTransmission</type>
         <joint name="roll_joint">
-            <hardwareInterface>hardware_interface/EffortJointInterface</hardwareInterface>
+            <hardwareInterface>hardware_interface/PositionJointInterface</hardwareInterface>
         </joint>
         <actuator name="roll_joint_motor">
-            <hardwareInterface>hardware_interface/EffortJointInterface</hardwareInterface>
+            <hardwareInterface>hardware_interface/PositionJointInterface</hardwareInterface>
             <mechanicalReduction>5</mechanicalReduction>
         </actuator>
@@ -174,8 +174,8 @@
         <type>transmission_interface/SimpleTransmission</type>
         <joint name="yaw_joint">
-            <hardwareInterface>hardware_interface/EffortJointInterface</hardwareInterface>
+            <hardwareInterface>hardware_interface/PositionJointInterface</hardwareInterface>
         </joint>
         <actuator name="yaw_joint_motor">
-            <hardwareInterface>hardware_interface/EffortJointInterface</hardwareInterface>
+            <hardwareInterface>hardware_interface/PositionJointInterface</hardwareInterface>
             <mechanicalReduction>5</mechanicalReduction>
         </actuator>
@@ -184,8 +184,8 @@
         <type>transmission_interface/SimpleTransmission</type>
         <joint name="roll_2_joint">
-            <hardwareInterface>hardware_interface/EffortJointInterface</hardwareInterface>
+            <hardwareInterface>hardware_interface/PositionJointInterface</hardwareInterface>
         </joint>
         <actuator name="roll_2_joint_motor">
-            <hardwareInterface>hardware_interface/EffortJointInterface</hardwareInterface>
+            <hardwareInterface>hardware_interface/PositionJointInterface</hardwareInterface>
             <mechanicalReduction>5</mechanicalReduction>
         </actuator>
@@ -214,8 +214,8 @@
         <type>transmission_interface/SimpleTransmission</type>
         <joint name="left_finger_joint">
-            <hardwareInterface>hardware_interface/EffortJointInterface</hardwareInterface>
+            <hardwareInterface>hardware_interface/PositionJointInterface</hardwareInterface>
         </joint>
         <actuator name="left_finger_joint_motor">
-            <hardwareInterface>hardware_interface/EffortJointInterface</hardwareInterface>
+            <hardwareInterface>hardware_interface/PositionJointInterface</hardwareInterface>
             <mechanicalReduction>5</mechanicalReduction>
         </actuator>
@@ -224,8 +224,8 @@
         <type>transmission_interface/SimpleTransmission</type>
         <joint name="right_finger_joint">
-            <hardwareInterface>hardware_interface/EffortJointInterface</hardwareInterface>
+            <hardwareInterface>hardware_interface/PositionJointInterface</hardwareInterface>
         </joint>
         <actuator name="right_finger_joint_motor">
-            <hardwareInterface>hardware_interface/EffortJointInterface</hardwareInterface>
+            <hardwareInterface>hardware_interface/PositionJointInterface</hardwareInterface>
             <mechanicalReduction>5</mechanicalReduction>
         </actuator>
