Commit message: increasing linear joint limit

File: doris_description/urdf/doris_description.urdf.xacro (robot description, xacro)
@@ -65,5 +65,5 @@
         <origin xyz="0.20 0 0" rpy="0 0 0" />
         <axis xyz="0 0 1"/>
-        <limit effort="2000.0" lower="0.02" upper="0.5" velocity="0.5"/>
+        <limit effort="2000.0" lower="0.02" upper="0.6" velocity="0.5"/>
         <dynamics damping="0.5" friction="0.1"/>
     </joint>
@@ -134,8 +134,8 @@
         <type>transmission_interface/SimpleTransmission</type>
         <joint name="shoulder_joint">
-            <hardwareInterface>hardware_interface/PositionJointInterface</hardwareInterface>
+            <hardwareInterface>hardware_interface/EffortJointInterface</hardwareInterface>
         </joint>
         <actuator name="shoulder_joint_motor">
-            <hardwareInterface>hardware_interface/PositionJointInterface</hardwareInterface>
+            <hardwareInterface>hardware_interface/EffortJointInterface</hardwareInterface>
             <mechanicalReduction>5</mechanicalReduction>
         </actuator>
@@ -144,8 +144,8 @@
         <type>transmission_interface/SimpleTransmission</type>
         <joint name="forearm_shoulder_joint">
-            <hardwareInterface>hardware_interface/PositionJointInterface</hardwareInterface>
+            <hardwareInterface>hardware_interface/EffortJointInterface</hardwareInterface>
         </joint>
         <actuator name="forearm_shoulder_joint_motor">
-            <hardwareInterface>hardware_interface/PositionJointInterface</hardwareInterface>
+            <hardwareInterface>hardware_interface/EffortJointInterface</hardwareInterface>
             <mechanicalReduction>5</mechanicalReduction>
         </actuator>
@@ -154,8 +154,8 @@
         <type>transmission_interface/SimpleTransmission</type>
         <joint name="elbow_joint">
-            <hardwareInterface>hardware_interface/PositionJointInterface</hardwareInterface>
+            <hardwareInterface>hardware_interface/EffortJointInterface</hardwareInterface>
         </joint>
         <actuator name="elbow_joint_motor">
-            <hardwareInterface>hardware_interface/PositionJointInterface</hardwareInterface>
+            <hardwareInterface>hardware_interface/EffortJointInterface</hardwareInterface>
             <mechanicalReduction>5</mechanicalReduction>
         </actuator>
@@ -164,8 +164,8 @@
         <type>transmission_interface/SimpleTransmission</type>
         <joint name="roll_joint">
-            <hardwareInterface>hardware_interface/PositionJointInterface</hardwareInterface>
+            <hardwareInterface>hardware_interface/EffortJointInterface</hardwareInterface>
         </joint>
         <actuator name="roll_joint_motor">
-            <hardwareInterface>hardware_interface/PositionJointInterface</hardwareInterface>
+            <hardwareInterface>hardware_interface/EffortJointInterface</hardwareInterface>
             <mechanicalReduction>5</mechanicalReduction>
         </actuator>
@@ -174,8 +174,8 @@
         <type>transmission_interface/SimpleTransmission</type>
         <joint name="yaw_joint">
-            <hardwareInterface>hardware_interface/PositionJointInterface</hardwareInterface>
+            <hardwareInterface>hardware_interface/EffortJointInterface</hardwareInterface>
         </joint>
         <actuator name="yaw_joint_motor">
-            <hardwareInterface>hardware_interface/PositionJointInterface</hardwareInterface>
+            <hardwareInterface>hardware_interface/EffortJointInterface</hardwareInterface>
             <mechanicalReduction>5</mechanicalReduction>
         </actuator>
@@ -184,8 +184,8 @@
         <type>transmission_interface/SimpleTransmission</type>
         <joint name="roll_2_joint">
-            <hardwareInterface>hardware_interface/PositionJointInterface</hardwareInterface>
+            <hardwareInterface>hardware_interface/EffortJointInterface</hardwareInterface>
         </joint>
         <actuator name="roll_2_joint_motor">
-            <hardwareInterface>hardware_interface/PositionJointInterface</hardwareInterface>
+            <hardwareInterface>hardware_interface/EffortJointInterface</hardwareInterface>
             <mechanicalReduction>5</mechanicalReduction>
         </actuator>
@@ -214,8 +214,8 @@
         <type>transmission_interface/SimpleTransmission</type>
         <joint name="left_finger_joint">
-            <hardwareInterface>hardware_interface/PositionJointInterface</hardwareInterface>
+            <hardwareInterface>hardware_interface/EffortJointInterface</hardwareInterface>
         </joint>
         <actuator name="left_finger_joint_motor">
-            <hardwareInterface>hardware_interface/PositionJointInterface</hardwareInterface>
+            <hardwareInterface>hardware_interface/EffortJointInterface</hardwareInterface>
             <mechanicalReduction>5</mechanicalReduction>
         </actuator>
@@ -224,8 +224,8 @@
         <type>transmission_interface/SimpleTransmission</type>
         <joint name="right_finger_joint">
-            <hardwareInterface>hardware_interface/PositionJointInterface</hardwareInterface>
+            <hardwareInterface>hardware_interface/EffortJointInterface</hardwareInterface>
         </joint>
         <actuator name="right_finger_joint_motor">
-            <hardwareInterface>hardware_interface/PositionJointInterface</hardwareInterface>
+            <hardwareInterface>hardware_interface/EffortJointInterface</hardwareInterface>
             <mechanicalReduction>5</mechanicalReduction>
         </actuator>

Commit message: add gripper range sensor

File: doris_description/urdf/doris_description.urdf.xacro (robot description, xacro)
@@ -15,4 +15,10 @@
         <child link="base_link" />
         <parent link="base_footprint" />
+    </joint>
+    <link name="gripper_ir_link"></link>
+    <joint name="gripper_ir_joint" type="fixed">
+        <child link="gripper_ir_link"/>
+        <parent link="gripper_link"/>
+        <origin xyz="0.05 0 -0.05" rpy="0 1.57 0"/>
     </joint>
     <link name="frontal_caster_link">
@@ -114,8 +120,8 @@
         <type>transmission_interface/SimpleTransmission</type>
         <joint name="dorso_arm_base">
-            <hardwareInterface>hardware_interface/PositionJointInterface</hardwareInterface>
+            <hardwareInterface>hardware_interface/EffortJointInterface</hardwareInterface>
         </joint>
         <actuator name="dorso_arm_linear_actuator">
-            <hardwareInterface>hardware_interface/PositionJointInterface</hardwareInterface>
+            <hardwareInterface>hardware_interface/EffortJointInterface</hardwareInterface>
             <mechanicalReduction>1</mechanicalReduction>
         </actuator>
@@ -134,8 +140,8 @@
         <type>transmission_interface/SimpleTransmission</type>
         <joint name="shoulder_joint">
-            <hardwareInterface>hardware_interface/PositionJointInterface</hardwareInterface>
+            <hardwareInterface>hardware_interface/EffortJointInterface</hardwareInterface>
         </joint>
         <actuator name="shoulder_joint_motor">
-            <hardwareInterface>hardware_interface/PositionJointInterface</hardwareInterface>
+            <hardwareInterface>hardware_interface/EffortJointInterface</hardwareInterface>
             <mechanicalReduction>5</mechanicalReduction>
         </actuator>
@@ -144,8 +150,8 @@
         <type>transmission_interface/SimpleTransmission</type>
         <joint name="forearm_shoulder_joint">
-            <hardwareInterface>hardware_interface/PositionJointInterface</hardwareInterface>
+            <hardwareInterface>hardware_interface/EffortJointInterface</hardwareInterface>
         </joint>
         <actuator name="forearm_shoulder_joint_motor">
-            <hardwareInterface>hardware_interface/PositionJointInterface</hardwareInterface>
+            <hardwareInterface>hardware_interface/EffortJointInterface</hardwareInterface>
             <mechanicalReduction>5</mechanicalReduction>
         </actuator>
@@ -154,8 +160,8 @@
         <type>transmission_interface/SimpleTransmission</type>
         <joint name="elbow_joint">
-            <hardwareInterface>hardware_interface/PositionJointInterface</hardwareInterface>
+            <hardwareInterface>hardware_interface/EffortJointInterface</hardwareInterface>
         </joint>
         <actuator name="elbow_joint_motor">
-            <hardwareInterface>hardware_interface/PositionJointInterface</hardwareInterface>
+            <hardwareInterface>hardware_interface/EffortJointInterface</hardwareInterface>
             <mechanicalReduction>5</mechanicalReduction>
         </actuator>
@@ -164,8 +170,8 @@
         <type>transmission_interface/SimpleTransmission</type>
         <joint name="roll_joint">
-            <hardwareInterface>hardware_interface/PositionJointInterface</hardwareInterface>
+            <hardwareInterface>hardware_interface/EffortJointInterface</hardwareInterface>
         </joint>
         <actuator name="roll_joint_motor">
-            <hardwareInterface>hardware_interface/PositionJointInterface</hardwareInterface>
+            <hardwareInterface>hardware_interface/EffortJointInterface</hardwareInterface>
             <mechanicalReduction>5</mechanicalReduction>
         </actuator>
@@ -174,8 +180,8 @@
         <type>transmission_interface/SimpleTransmission</type>
         <joint name="yaw_joint">
-            <hardwareInterface>hardware_interface/PositionJointInterface</hardwareInterface>
+            <hardwareInterface>hardware_interface/EffortJointInterface</hardwareInterface>
         </joint>
         <actuator name="yaw_joint_motor">
-            <hardwareInterface>hardware_interface/PositionJointInterface</hardwareInterface>
+            <hardwareInterface>hardware_interface/EffortJointInterface</hardwareInterface>
             <mechanicalReduction>5</mechanicalReduction>
         </actuator>
@@ -184,8 +190,8 @@
         <type>transmission_interface/SimpleTransmission</type>
         <joint name="roll_2_joint">
-            <hardwareInterface>hardware_interface/PositionJointInterface</hardwareInterface>
+            <hardwareInterface>hardware_interface/EffortJointInterface</hardwareInterface>
         </joint>
         <actuator name="roll_2_joint_motor">
-            <hardwareInterface>hardware_interface/PositionJointInterface</hardwareInterface>
+            <hardwareInterface>hardware_interface/EffortJointInterface</hardwareInterface>
             <mechanicalReduction>5</mechanicalReduction>
         </actuator>
@@ -214,8 +220,8 @@
         <type>transmission_interface/SimpleTransmission</type>
         <joint name="left_finger_joint">
-            <hardwareInterface>hardware_interface/PositionJointInterface</hardwareInterface>
+            <hardwareInterface>hardware_interface/EffortJointInterface</hardwareInterface>
         </joint>
         <actuator name="left_finger_joint_motor">
-            <hardwareInterface>hardware_interface/PositionJointInterface</hardwareInterface>
+            <hardwareInterface>hardware_interface/EffortJointInterface</hardwareInterface>
             <mechanicalReduction>5</mechanicalReduction>
         </actuator>
@@ -224,8 +230,8 @@
         <type>transmission_interface/SimpleTransmission</type>
         <joint name="right_finger_joint">
-            <hardwareInterface>hardware_interface/PositionJointInterface</hardwareInterface>
+            <hardwareInterface>hardware_interface/EffortJointInterface</hardwareInterface>
         </joint>
         <actuator name="right_finger_joint_motor">
-            <hardwareInterface>hardware_interface/PositionJointInterface</hardwareInterface>
+            <hardwareInterface>hardware_interface/EffortJointInterface</hardwareInterface>
             <mechanicalReduction>5</mechanicalReduction>
         </actuator>
@@ -378,4 +384,41 @@
         </plugin>
     </gazebo>
+    <gazebo reference="gripper_ir_link">
+        <sensor type="ray" name="ir_gripper">
+            <pose>0 0 0 0 0 0</pose>
+            <update_rate>50</update_rate>
+            <ray>
+                <scan>
+                    <horizontal>
+                        <samples>1</samples>
+                        <resolution>1.0</resolution>
+                        <min_angle>-0.01</min_angle>
+                        <max_angle>0.01</max_angle>
+                    </horizontal>
+                    <vertical>
+                        <samples>1</samples>
+                        <resolution>1</resolution>
+                        <min_angle>-0.01</min_angle>
+                        <max_angle>0.01</max_angle>
+                    </vertical>
+                </scan>
+                <range>
+                    <min>0.01</min>
+                    <max>1.5</max>
+                    <resolution>0.02</resolution>
+                </range>
+            </ray>
+            <plugin filename="libgazebo_ros_range.so" name="gazebo_ros_range">
+                <gaussianNoise>0.005</gaussianNoise>
+                <alwaysOn>true</alwaysOn>
+                <updateRate>5</updateRate>
+                <topicName>/gripper/range</topicName>
+                <frameName>ir_gripper</frameName>
+                <visualize>false</visualize>
+                <radiation>infrared</radiation>
+                <fov>0.02</fov>
+            </plugin>
+        </sensor>
+    </gazebo>
     <!--
     <gazebo reference="doris_hand">

Commit message: moving hokuyo

File: doris_description/urdf/doris_description.urdf.xacro (robot description, xacro)
@@ -104,6 +104,6 @@
         <origin xyz="-0.25 -0.7 0.01" rpy="${3.1416/2} ${-3.1416/2} 3.1416" />
     </joint-->
-    <xacro:hokuyo_utm30lx name="hokuyo" parent="base_link" ros_topic="scan2" update_rate="30" ray_count="500" min_angle="0" max_angle="-180">
-        <origin xyz="0.32 0 0" rpy="3.14 0 0" />
+    <xacro:hokuyo_utm30lx name="hokuyo" parent="base_link" ros_topic="scan2" update_rate="30" ray_count="500" min_angle="-90" max_angle="90">
+        <origin xyz="0.32 0 0.08" rpy="3.14 0 0" />
     </xacro:hokuyo_utm30lx>
     <transmission name="trans_left_wheel_joint">
@@ -367,5 +367,5 @@
         <min_depth>0.1</min_depth>
     </gazebo>
-    <gazebo>
+    <!--gazebo>
         <plugin name="gazebo_grasp_fix" filename="libgazebo_grasp_fix.so">
             <arm>
@@ -383,5 +383,5 @@
             <contact_topic>__default_topic__</contact_topic>
         </plugin>
-    </gazebo>
+    </gazebo-->
     <gazebo reference="gripper_ir_link">
         <sensor type="ray" name="ir_gripper">

Commit message: larc 2021

File: doris_description/urdf/doris_description.urdf.xacro (robot description, xacro)
@@ -20,5 +20,5 @@
         <child link="gripper_ir_link"/>
         <parent link="gripper_link"/>
-        <origin xyz="0.05 0 -0.05" rpy="0 1.57 0"/>
+        <origin xyz="0.02 0 -0.01" rpy="0 1.57 0"/>
     </joint>
     <link name="frontal_caster_link">
@@ -105,5 +105,5 @@
     </joint-->
     <xacro:hokuyo_utm30lx name="hokuyo" parent="base_link" ros_topic="scan2" update_rate="30" ray_count="500" min_angle="-90" max_angle="90">
-        <origin xyz="0.32 0 0.08" rpy="3.14 0 0" />
+        <origin xyz="0.32 0 0" rpy="3.14 0 0" />
     </xacro:hokuyo_utm30lx>
     <transmission name="trans_left_wheel_joint">
@@ -378,10 +378,10 @@
             <update_rate>4</update_rate>
             <grip_count_threshold>4</grip_count_threshold>
-            <max_grip_count>8</max_grip_count>
+            <max_grip_count>4</max_grip_count>
             <release_tolerance>0.005</release_tolerance>
             <disable_collisions_on_attach>false</disable_collisions_on_attach>
             <contact_topic>__default_topic__</contact_topic>
         </plugin>
-    </gazebo-->
+    </gazeb-->
     <gazebo reference="gripper_ir_link">
         <sensor type="ray" name="ir_gripper">
@@ -410,4 +410,5 @@
             </ray>
             <plugin filename="libgazebo_ros_range.so" name="gazebo_ros_range">
+                <selfCollide>false</selfCollide>
                 <alwaysOn>true</alwaysOn>
                 <updateRate>5</updateRate>
@@ -420,4 +421,32 @@
         </sensor>
     </gazebo>
+    <gazebo reference="left_finger_link">
+        <sensor name="left_finger_bumper" type="contact">
+            <selfCollide>false</selfCollide>
+            <alwaysOn>true</alwaysOn>
+            <updateRate>50.0</updateRate>
+            <contact>
+                <collision>left_finger_link_collision</collision>
+            </contact>
+            <plugin name="left_finger_ros_bumper_controller" filename="libgazebo_ros_bumper.so">
+                <bumperTopicName>/gripper/contact/left</bumperTopicName>
+                <frameName>world</frameName>
+            </plugin>
+        </sensor>
+    </gazebo>
+    <gazebo reference="right_finger_link">
+        <sensor name="right_finger_bumper" type="contact">
+            <selfCollide>false</selfCollide>
+            <alwaysOn>true</alwaysOn>
+            <updateRate>50.0</updateRate>
+            <contact>
+                <collision>right_finger_link_collision</collision>
+            </contact>
+            <plugin name="right_finger_ros_bumper_controller" filename="libgazebo_ros_bumper.so">
+                <bumperTopicName>/gripper/contact/right</bumperTopicName>
+                <frameName>world</frameName>
+            </plugin>
+        </sensor>
+    </gazebo>
     <!--
     <gazebo reference="doris_hand">
