Commit message: Add urdf of robot without arm

File: doris_description/urdf/doris_description.urdf.xacro (robot description, xacro)
@@ -1,66 +1,5 @@
 <?xml version="1.0"?>
 <robot xmlns:xacro="http://www.ros.org/wiki/xacro" name="doris">
-    <xacro:include filename="$(find patrolbot_description)/urdf/patrolbot_description.urdf" />
-    <!--xacro:include filename="$(find doris_arm_description)/urdf/doris_arm_description.urdf.xacro" /-->
-    <!--xacro:include filename="$(find interbotix_xsarm_descriptions)/urdf/doris_arm.urdf.xacro" /-->
-    <!--xacro:include filename="$(find doris_arm_description)/urdf/hand.xacro" /-->
-    <xacro:include filename="$(find doris_dorso_description)/urdf/doris_dorso_description.urdf" />
-    <!--xacro:include filename="$(find kinect2_description)/urdf/kinect2_description.urdf.xacro" /-->
-    <xacro:include filename="$(find doris_head_description)/urdf/doris_head.urdf" />
-    <xacro:include filename="$(find doris_sensors_description)/urdf/hokuyo.urdf.xacro" />
-    <xacro:include filename="$(find doris_sensors_description)/urdf/sick_lms1xx.urdf.xacro" />
-    <xacro:include filename="$(find doris_sensors_description)/urdf/materials.xacro" />
-    <xacro:include filename="$(find doris_sensors_description)/urdf/kinect_camera.urdf.xacro" />
-    <xacro:include filename="$(find hector_sensors_description)/urdf/realsense_d435_camera.urdf.xacro" />
-    <!--xacro:include filename="$(find lms1xx)/urdf/sick_lms1xx.urdf.xacro" /-->
-    <link name="base_footprint"></link>
-    <joint name="base_joint" type="fixed">
-        <child link="base_link" />
-        <parent link="base_footprint" />
-    </joint>
-    <link name="frontal_caster_link">
-        <inertial>
-            <origin xyz="0 0 0" rpy="0 0 0" />
-            <mass value="0.1" />
-            <inertia ixx="0.001" ixy="0" ixz="0" iyy="0.001" iyz="0" izz="0.001" />
-        </inertial>
-        <collision>
-            <origin xyz="0 0 0" rpy="0 0 0" />
-            <geometry>
-                <sphere radius="0.05"/>
-            </geometry>
-        </collision>
-    </link>
-    <joint name="frontal_caster_joint" type="fixed">
-        <parent link="base_link" />
-        <child link="frontal_caster_link" />
-        <origin xyz="0.2 0 0" rpy="0 0 0" />
-    </joint>
-    <link name="rear_caster_link">
-        <inertial>
-            <origin xyz="0 0 0" rpy="0 0 0" />
-            <mass value="0.1" />
-            <inertia ixx="0.001" ixy="0" ixz="0" iyy="0.001" iyz="0" izz="0.001" />
-        </inertial>
-        <collision>
-            <origin xyz="0 0 0" rpy="0 0 0" />
-            <geometry>
-                <sphere radius="0.05"/>
-            </geometry>
-        </collision>
-    </link>
-    <joint name="rear_caster_joint" type="fixed">
-        <parent link="base_link" />
-        <child link="rear_caster_link" />
-        <origin xyz="-0.2 0 0" rpy="0 0 0" />
-    </joint>
-    <!--
-    <xacro:hand ns="doris" rpy="0 0 1.570" xyz="0 0 0.1" connected_to="roll_2_link" safety_distance="0.00" use_cylinder_collision_model="false" />
-    -->
-    <joint name="base_link_dorso" type="fixed">
-        <parent link="base_link" />
-        <child link="dorso_link" />
-        <origin xyz="0 0 0.28" rpy="0 0 0" />
-    </joint>
+    <xacro:include filename="$(find doris_description)/urdf/doris_no_arm.urdf.xacro" />
     <joint name="dorso_arm_base" type="fixed">
         <parent link="dorso_link" />
@@ -68,124 +7,3 @@
         <origin xyz="0.20 0 0.1" rpy="0 0 0" />
     </joint>
-    <xacro:sick_lms1xx />
-    <joint name="laser_joint" type="fixed">
-        <origin xyz="0.222 0 -0.07" rpy="0 0 0" />
-        <parent link="dorso_link" />
-        <child link="laser" />
-    </joint>
-    <!--joint name="dorso_kinect" type="fixed">
-        <parent link="dorso_link" />
-        <child link="kinect_link" />
-        <origin xyz="-0.18 0 0.01" rpy="0 ${3.1416/2} 3.1416" />
-    </joint-->
-    <!--xacro:sensor_kinect prefix="" name="kinect" parent="dorso_link" cam_px="-0.18" cam_py="0" cam_pz="0.01" cam_or="${-3.1416/2}" cam_op="0" cam_oy="${3.1416/2}"></xacro:sensor_kinect-->
-    <xacro:kinect_camera name="kinect2" parent="dorso_link">
-        <origin xyz="0.23 0 0.82" rpy="0 0 0" />
-    </xacro:kinect_camera>
-    <!--
-    <xacro:realsense_d435_camera_with_mount name="realsense" parent="roll_2_link">
-        <origin xyz="0 0.03 0.1" rpy="-1.570 -1.570 0" />
-    </xacro:realsense_d435_camera_with_mount>
-    -->
-    <joint name="dorso_head" type="fixed">
-        <parent link="dorso_link" />
-        <child link="head_root" />
-        <origin xyz="0 0 1.16" rpy="0 0 0" />
-    </joint>
-    <!--joint name="dorso_hokuyo" type="fixed">
-        <parent link="dorso_link" />
-        <child link="hokuyo_link" />
-        <origin xyz="-0.25 -0.7 0.01" rpy="${3.1416/2} ${-3.1416/2} 3.1416" />
-    </joint-->
-    <!--xacro:hokuyo_utm30lx name="hokuyo" parent="base_link" ros_topic="scan2" update_rate="30" ray_count="500" min_angle="-90" max_angle="90">
-        <origin xyz="0.32 0 0" rpy="3.14 0 0" />
-    </xacro:hokuyo_utm30lx-->
-    <xacro:sensor_hokuyo parent="base_link" xyz="0.2 0 0" rpy="0 3.1416 3.1416" />
-    <transmission name="trans_left_wheel_joint">
-        <type>transmission_interface/SimpleTransmission</type>
-        <joint name="left_wheel_joint">
-            <hardwareInterface>hardware_interface/EffortJointInterface</hardwareInterface>
-        </joint>
-        <actuator name="left_wheel_joint_motor">
-            <hardwareInterface>hardware_interface/EffortJointInterface</hardwareInterface>
-            <mechanicalReduction>1</mechanicalReduction>
-        </actuator>
-    </transmission>
-    <transmission name="trans_right_wheel_joint">
-        <type>transmission_interface/SimpleTransmission</type>
-        <joint name="right_wheel_joint">
-            <hardwareInterface>hardware_interface/EffortJointInterface</hardwareInterface>
-        </joint>
-        <actuator name="right_wheel_joint_motor">
-            <hardwareInterface>hardware_interface/EffortJointInterface</hardwareInterface>
-            <mechanicalReduction>1</mechanicalReduction>
-        </actuator>
-    </transmission>
-    <gazebo>
-        <plugin name="differential_drive_controller" filename="libgazebo_ros_diff_drive.so">
-            <!-- Plugin update rate in Hz -->
-            <updateRate>50</updateRate>
-            <!-- Name of left joint, defaults to `left_joint` -->
-            <leftJoint>left_wheel_joint</leftJoint>
-            <!-- Name of right joint, defaults to `right_joint` -->
-            <rightJoint>right_wheel_joint</rightJoint>
-            <!-- The distance from the center of one wheel to the other, in meters, defaults to 0.34 m -->
-            <wheelSeparation>0.31</wheelSeparation>
-            <!-- Diameter of the wheels, in meters, defaults to 0.15 m -->
-            <wheelDiameter>0.2</wheelDiameter>
-            <!-- Wheel acceleration, in rad/s^2, defaults to 0.0 rad/s^2 -->
-            <wheelAcceleration>1.0</wheelAcceleration>
-            <!-- Maximum torque which the wheels can produce, in Nm, defaults to 5 Nm -->
-            <wheelTorque>200</wheelTorque>
-            <!-- Topic to receive geometry_msgs/Twist message commands, defaults to `cmd_vel` -->
-            <commandTopic>cmd_vel</commandTopic>
-            <!-- Topic to publish nav_msgs/Odometry messages, defaults to `odom` -->
-            <odometryTopic>odom</odometryTopic>
-            <!-- Odometry frame, defaults to `odom` -->
-            <odometryFrame>odom</odometryFrame>
-            <!-- Robot frame to calculate odometry from, defaults to `base_footprint` -->
-            <robotBaseFrame>base_footprint</robotBaseFrame>
-            <!-- Odometry source, 0 for ENCODER, 1 for WORLD, defaults to WORLD -->
-            <odometrySource>1</odometrySource>
-            <!-- Set to true to publish transforms for the wheel links, defaults to false -->
-            <publishWheelTF>false</publishWheelTF>
-            <!-- Set to true to publish transforms for the odometry, defaults to true -->
-            <publishOdom>true</publishOdom>
-            <!-- Set to true to publish sensor_msgs/JointState on /joint_states for the wheel joints, defaults to false -->
-            <publishWheelJointState>false</publishWheelJointState>
-            <!-- Set to true to swap right and left wheels, defaults to true -->
-            <legacyMode>false</legacyMode>
-            <robotNamespace>/</robotNamespace>
-        </plugin>
-    </gazebo>
-    <material name="gray_material">
-        <color rgba="0.5 0.5 0.5 1.0" />
-    </material>
-    <material name="black_material">
-        <color rgba="0.1 0.1 0.1 1.0" />
-    </material>
-    <gazebo reference="base_link">
-        <material>Gazebo/Gray</material>
-    </gazebo>
-    <gazebo reference="left_wheel_link">
-        <material>Gazebo/DarkGray</material>
-        <mu1>0.95</mu1>
-        <mu2>0.95</mu2>
-    </gazebo>
-    <gazebo reference="right_wheel_link">
-        <material>Gazebo/DarkGray</material>
-        <mu1>0.95</mu1>
-        <mu2>0.95</mu2>
-    </gazebo>
-    <gazebo reference="frontal_caster_link">
-        <mu1>0.000001</mu1>
-        <mu2>0.000001</mu2>
-    </gazebo>
-    <gazebo reference="rear_caster_link">
-        <mu1>0.000001</mu1>
-        <mu2>0.000001</mu2>
-    </gazebo>
-    <gazebo reference="dorso_link">
-        <material>Gazebo/DarkGray</material>
-    </gazebo>
 </robot>

Commit message: Update robot urdf.

File: doris_description/urdf/doris_description.urdf.xacro (robot description, xacro)
@@ -5,5 +5,5 @@
         <parent link="dorso_link" />
         <child link="doris_arm/base_link" />
-        <origin xyz="0.20 0 0.1" rpy="0 0 0" />
+        <origin xyz="0.25 0 0.35" rpy="0 0 0" />
     </joint>
 </robot>

File: doris_description/urdf/doris_no_arm.urdf.xacro (robot description, xacro)
@@ -61,9 +61,9 @@
         <parent link="base_link" />
         <child link="dorso_link" />
-        <origin xyz="0 0 0.28" rpy="0 0 0" />
+        <origin xyz="0 0 0.36" rpy="0 0 0" />
     </joint>
     <xacro:sick_lms1xx />
     <joint name="laser_joint" type="fixed">
-        <origin xyz="0.222 0 -0.07" rpy="0 0 0" />
+        <origin xyz="0.222 0 0.12" rpy="0 0 0" />
         <parent link="dorso_link" />
         <child link="laser" />
@@ -76,5 +76,5 @@
     <!--xacro:sensor_kinect prefix="" name="kinect" parent="dorso_link" cam_px="-0.18" cam_py="0" cam_pz="0.01" cam_or="${-3.1416/2}" cam_op="0" cam_oy="${3.1416/2}"></xacro:sensor_kinect-->
     <xacro:kinect_camera name="kinect2" parent="dorso_link">
-        <origin xyz="0.23 0 0.82" rpy="0 0 0" />
+        <origin xyz="0.2 0 0.82" rpy="0 0 0" />
     </xacro:kinect_camera>
     <!--
@@ -86,5 +86,5 @@
         <parent link="dorso_link" />
         <child link="head_root" />
-        <origin xyz="0 0 1.16" rpy="0 0 0" />
+        <origin xyz="0 0 0.9" rpy="0 0 0" />
     </joint>
     <!--joint name="dorso_hokuyo" type="fixed">

File: doris_dorso_description/urdf/doris_dorso_description.urdf (robot description, URDF)
Before this commit: robot doris_dorso_description, 1 links, 0 joints
Links:
- link dorso_link: geometry collision mesh filename=package://doris_dorso_description/meshes/dorso_link.STL scale=0.001 0.001 0.001; visual mesh filename=package://doris_dorso_description/meshes/dorso_link.STL scale=0.001 0.001 0.001

File: patrolbot_description/urdf/patrolbot_description.urdf (robot description, URDF)
Before this commit: robot patrolbot_description, 3 links, 2 joints
Links:
- link base_link: geometry collision mesh filename=package://patrolbot_description/meshes/hull.stl scale=1 1 1; visual mesh filename=package://patrolbot_description/meshes/hull.stl scale=1 1 1
