Commit message: some modifications to work on doris

File: doris_description/urdf/doris_no_arm.urdf.xacro (robot description, xacro)
@@ -67,5 +67,5 @@
         <origin xyz="0.222 0 -0.07" rpy="0 0 0" />
         <parent link="dorso_link" />
-        <child link="laser" />
+        <child link="sick_link" />
     </joint>
     <!--joint name="dorso_kinect" type="fixed">

File: doris_sensors_description/urdf/sick_lms1xx.urdf.xacro (robot description, xacro)
@@ -26,5 +26,5 @@
 -->
 <robot xmlns:xacro="http://www.ros.org/wiki/xacro">
-  <xacro:macro name="sick_lms1xx" params="frame:=laser topic:=scan sample_size:=720 update_rate:=50
+  <xacro:macro name="sick_lms1xx" params="frame:=sick_link topic:=scan sample_size:=720 update_rate:=50
                min_angle:=-1.570 max_angle:=1.570 min_range:=0.1 max_range:=30.0 robot_namespace:=/" >
     <link name="${frame}">

Commit message: move kinect working

File: doris_description/urdf/doris_no_arm.urdf.xacro (robot description, xacro)
@@ -74,12 +74,7 @@
         <origin xyz="0.1362 0 0.8465" rpy="0 0 0" />
     </joint-->
-    <!--joint name="dorso_kinect" type="fixed">
-        <parent link="dorso_link" />
-        <child link="kinect_link" />
-        <origin xyz="-0.18 0 0.01" rpy="0 ${3.1416/2} 3.1416" />
-    </joint-->
-    <!--xacro:sensor_kinect prefix="" name="kinect" parent="dorso_link" cam_px="-0.18" cam_py="0" cam_pz="0.01" cam_or="${-3.1416/2}" cam_op="0" cam_oy="${3.1416/2}"></xacro:sensor_kinect-->
+    <!-- <xacro:sensor_kinect prefix="" name="kinect" parent="dorso_link" cam_px="-0.18" cam_py="0" cam_pz="0.01" cam_or="${-3.1416/2}" cam_op="0" cam_oy="${3.1416/2}"></xacro:sensor_kinect--> -->
     <xacro:kinect_camera name="kinect2" parent="dorso_link">
-        <origin xyz="0.1362 0 0.8465" rpy="0 0 0" />
+        <origin xyz="0.1362 0 0.8465" rpy="-1.57 0 -1.57" />
     </xacro:kinect_camera>
     <!--
@@ -88,4 +83,9 @@
     </xacro:realsense_d435_camera_with_mount>
     -->
+    <!-- <joint name="dorso_kinect" type="fixed">
+        <parent link="dorso_link" />
+        <child link="kinect2_root" />
+        <origin xyz="-0.0767 0 0.81" rpy="0 0 0" />
+    </joint> -->
     <joint name="dorso_head" type="fixed">
         <parent link="dorso_link" />

File: doris_sensors_description/urdf/kinect_camera.urdf.xacro (robot description, xacro)
@@ -4,14 +4,20 @@
     <xacro:property name="M_PI" value="3.1415926535897931"/>
     <xacro:macro name="kinect_camera_model" params="name parent *origin">
-      <joint name="${name}_joint" type="continuous">
+      <joint name="kinect2_joint" type="continuous">
+        <parent link="${parent}" />
+        <child link="${name}_link" />
+        <origin xyz="0.1362 0 0.8465" rpy="-1.57 0 -1.57" />
+        <axis xyz="0 -1 0" />
+      </joint>
+      <!-- <joint name="${name}_joint" type="continuous">
         <xacro:insert_block name="origin"/>
         <parent link="${parent}"/>
         <child link="${name}_link"/>
         <axis xyz="1 0 0" />
-      </joint>
+      </joint> -->
       <link name="${name}_link">
         <xacro:inertial_sphere mass="0.01" diameter="0.07" />
         <visual>
-          <origin xyz="0 0 0" rpy="0 0 0" />
+          <origin xyz="0 0 0" rpy="0 -1.57 -1.57" />
           <geometry>
             <mesh filename="package://hector_sensors_description/meshes/kinect_camera/kinect_camera_simple.dae"/>

Commit message: adding realsense with pan and tilt angles

File: doris_description/urdf/doris_no_arm.urdf.xacro (robot description, xacro)
@@ -7,4 +7,5 @@
     <xacro:include filename="$(find doris_dorso_description)/urdf/doris_dorso_description.urdf" />
     <!--xacro:include filename="$(find kinect2_description)/urdf/kinect2_description.urdf.xacro" /-->
+    <!--xacro:include filename="$(find kinect2_description)/urdf/kinect2_description.urdf.xacro" /-->
     <xacro:include filename="$(find doris_head_description)/urdf/doris_head.urdf" />
     <xacro:include filename="$(find doris_sensors_description)/urdf/hokuyo.urdf.xacro" />
@@ -12,5 +13,7 @@
     <xacro:include filename="$(find doris_sensors_description)/urdf/materials.xacro" />
     <xacro:include filename="$(find doris_sensors_description)/urdf/kinect_camera.urdf.xacro" />
+    <xacro:include filename="$(find doris_sensors_description)/urdf/realsense_camera.urdf.xacro" />
     <xacro:include filename="$(find hector_sensors_description)/urdf/realsense_d435_camera.urdf.xacro" />
+    <!-- <xacro:include filename="$(find realsense2_description)/urdf/_d435.urdf.xacro" /> -->
     <!--xacro:include filename="$(find lms1xx)/urdf/sick_lms1xx.urdf.xacro" /-->
     <link name="base_footprint"></link>
@@ -74,7 +77,16 @@
         <origin xyz="0.1362 0 0.8465" rpy="0 0 0" />
     </joint-->
+    <xacro:realsense_camera name="camera" parent="dorso_link">
+        <origin xyz="0.095 0 0.8" rpy="0 0 0" />
+    </xacro:realsense_camera>
+    <!-- <link name="camera_link" />
+    <joint name="camera_joint" type="fixed">
+        <parent link="dorso_link"/>
+        <child link="camera_link"/>
+        <origin xyz="0.1362 0 0.8465" rpy="-1.57 0 -1.57"/>
+    </joint> -->
     <!-- <xacro:sensor_kinect prefix="" name="kinect" parent="dorso_link" cam_px="-0.18" cam_py="0" cam_pz="0.01" cam_or="${-3.1416/2}" cam_op="0" cam_oy="${3.1416/2}"></xacro:sensor_kinect--> -->
     <xacro:kinect_camera name="kinect2" parent="dorso_link">
-        <origin xyz="0.1362 0 0.8465" rpy="-1.57 0 -1.57" />
+        <origin xyz="0.1412 0 0.8465" rpy="-1.57 0 -1.57" />
     </xacro:kinect_camera>
     <!--

File: doris_sensors_description/urdf/kinect_camera.urdf.xacro (robot description, xacro)
@@ -18,10 +18,10 @@
       <link name="${name}_link">
         <xacro:inertial_sphere mass="0.01" diameter="0.07" />
-        <visual>
+        <!-- <visual>
           <origin xyz="0 0 0" rpy="0 -1.57 -1.57" />
           <geometry>
             <mesh filename="package://hector_sensors_description/meshes/kinect_camera/kinect_camera_simple.dae"/>
           </geometry>
-        </visual>
+        </visual> -->
         <collision>
           <origin xyz="0 0 0" rpy="0 0 0" />

Commit message: make realsense work in simulation

File: doris_description/urdf/doris_no_arm.urdf.xacro (robot description, xacro)
@@ -87,7 +87,7 @@
     </joint> -->
     <!-- <xacro:sensor_kinect prefix="" name="kinect" parent="dorso_link" cam_px="-0.18" cam_py="0" cam_pz="0.01" cam_or="${-3.1416/2}" cam_op="0" cam_oy="${3.1416/2}"></xacro:sensor_kinect--> -->
-    <xacro:kinect_camera name="kinect2" parent="dorso_link">
+    <!--xacro:kinect_camera name="kinect2" parent="dorso_link">
         <origin xyz="0.1412 0 0.8465" rpy="-1.57 0 -1.57" />
-    </xacro:kinect_camera>
+    </xacro:kinect_camera-->
     <!--
     <xacro:realsense_d435_camera_with_mount name="realsense" parent="roll_2_link">
@@ -135,4 +135,12 @@
     </transmission>
     <gazebo>
+        <plugin name="head_pan_mimic_joint" filename="libroboticsgroup_upatras_gazebo_mimic_joint_plugin.so">
+            <joint>head_pan_joint</joint>
+            <mimicJoint>horizontal_neck_joint</mimicJoint>
+        </plugin>
+        <plugin name="head_tilt_mimic_joint" filename="libroboticsgroup_upatras_gazebo_mimic_joint_plugin.so">
+            <joint>head_tilt_joint</joint>
+            <mimicJoint>vertical_neck_joint</mimicJoint>
+        </plugin>
         <plugin name="differential_drive_controller" filename="libgazebo_ros_diff_drive.so">
             <!-- Plugin update rate in Hz -->

File: doris_sensors_description/urdf/realsense_camera.urdf.xacro (robot description, xacro)
@@ -1,4 +1,5 @@
 <?xml version="1.0"?>
 <robot xmlns:xacro="http://www.ros.org/wiki/xacro">
+  <xacro:include filename="$(find doris_sensors_description)/urdf/realsense_d435_camera.urdf.xacro" />
   <xacro:property name="M_PI" value="3.1415926535897931"/>
   <xacro:macro name="realsense_camera" params="name parent *origin">
@@ -97,5 +98,5 @@
         </inertial>
       </link>
-      <link name="camera_link">
+      <!--link name="camera_link">
         <inertial>
             <origin rpy="0 0 0" xyz="-0.0132722976093535 0.00168171470080143 2.49829664994428E-06"/>
@@ -118,5 +119,8 @@
             </geometry>
         </collision>
-      </link>
+      </link-->
+      <xacro:realsense_d435_camera name="camera" parent="head_tilt_link">
+          <origin rpy="0 0 0" xyz="0.06705 0.0125 0"/>
+      </xacro:realsense_d435_camera>
       <joint name="camera_joint_static" type="fixed">
           <origin rpy="0 0 0" xyz="0.06705 0 -0.00425"/>
@@ -125,10 +129,37 @@
           <axis xyz="0 0 0"/>
       </joint>
-      <joint name="camera_joint" type="fixed">
+      <transmission name="trans_head_pan_joint">
+          <type>transmission_interface/SimpleTransmission</type>
+          <joint name="head_pan_joint">
+              <hardwareInterface>hardware_interface/EffortJointInterface</hardwareInterface>
+          </joint>
+          <actuator name="head_pan_joint_motor">
+              <hardwareInterface>hardware_interface/EffortJointInterface</hardwareInterface>
+              <mechanicalReduction>1</mechanicalReduction>
+          </actuator>
+      </transmission>
+      <transmission name="trans_head_tilt_joint">
+            <type>transmission_interface/SimpleTransmission</type>
+            <joint name="head_tilt_joint">
+                <hardwareInterface>hardware_interface/EffortJointInterface</hardwareInterface>
+            </joint>
+            <actuator name="head_tilt_joint_motor">
+                <hardwareInterface>hardware_interface/EffortJointInterface</hardwareInterface>
+                <mechanicalReduction>1</mechanicalReduction>
+            </actuator>
+        </transmission>
+      <gazebo>
+            <plugin name="gazebo_ros_control" filename="libgazebo_ros_control.so">
+                <robotSimType>gazebo_ros_control/DefaultRobotHWSim</robotSimType>
+                <legacyModeNS>true</legacyModeNS>
+                <robotNamespace>/doris_head</robotNamespace>
+            </plugin>
+        </gazebo>
+      <!--joint name="camera_joint" type="fixed">
           <origin rpy="0 0 0" xyz="0.06705 0 -0.00425"/>
           <parent link="head_tilt_link"/>
           <child link="camera_link"/>
           <axis xyz="0 0 0"/>
-      </joint>
+      </joint-->
       <!-- <xacro:sensor_d435 parent="head_tilt_link" use_nominal_extrinsics="false" add_plug="false" use_mesh="true">
           <origin xyz="0.06705 0 -0.00425" rpy="0 0 0"/>
