Commit message: removing arm from urdf

File: doris_description/urdf/doris.urdf.xacro (robot description, xacro)
@@ -5,5 +5,5 @@
         <parent link="dorso_link" />
         <child link="doris_arm/base_link" />
-        <origin xyz="0.25 0 0.35" rpy="0 0 0" />
+        <origin xyz="0.25 0 0.32" rpy="0 0 0" />
     </joint>
     <xacro:include filename="$(find doris_arm_description)/urdf/doris_arm.urdf.xacro" />

File: doris_description/urdf/doris_no_arm.urdf.xacro (robot description, xacro)
@@ -11,5 +11,5 @@
     <xacro:include filename="$(find doris_sensors_description)/urdf/sick_lms1xx.urdf.xacro" />
     <xacro:include filename="$(find doris_sensors_description)/urdf/materials.xacro" />
-    <xacro:include filename="$(find doris_sensors_description)/urdf/kinect_camera.urdf.xacro" />
+    <!--xacro:include filename="$(find doris_sensors_description)/urdf/kinect_camera.urdf.xacro" /-->
     <xacro:include filename="$(find hector_sensors_description)/urdf/realsense_d435_camera.urdf.xacro" />
     <!--xacro:include filename="$(find lms1xx)/urdf/sick_lms1xx.urdf.xacro" /-->
@@ -71,11 +71,16 @@
     <!--joint name="dorso_kinect" type="fixed">
         <parent link="dorso_link" />
+        <child link="kinect2_link" />
+        <origin xyz="0.1362 0 0.8465" rpy="0 0 0" />
+    </joint-->
+    <!--joint name="dorso_kinect" type="fixed">
+        <parent link="dorso_link" />
         <child link="kinect_link" />
         <origin xyz="-0.18 0 0.01" rpy="0 ${3.1416/2} 3.1416" />
     </joint-->
     <!--xacro:sensor_kinect prefix="" name="kinect" parent="dorso_link" cam_px="-0.18" cam_py="0" cam_pz="0.01" cam_or="${-3.1416/2}" cam_op="0" cam_oy="${3.1416/2}"></xacro:sensor_kinect-->
-    <xacro:kinect_camera name="kinect2" parent="dorso_link">
-        <origin xyz="0.2 0 0.82" rpy="0 0 0" />
-    </xacro:kinect_camera>
+    <!--xacro:kinect_camera name="kinect2" parent="dorso_link">
+        <origin xyz="0.1362 0 0.8465" rpy="0 0 0" />
+    </xacro:kinect_camera-->
     <!--
     <xacro:realsense_d435_camera_with_mount name="realsense" parent="roll_2_link">
@@ -86,5 +91,5 @@
         <parent link="dorso_link" />
         <child link="head_root" />
-        <origin xyz="0 0 0.9" rpy="0 0 0" />
+        <origin xyz="-0.0767 0 0.81" rpy="0 0 0" />
     </joint>
     <!--joint name="dorso_hokuyo" type="fixed">

Commit message: Add extra caster wheels to base urdf

File: doris_description/urdf/doris.urdf.xacro (robot description, xacro)
@@ -2,4 +2,5 @@
 <robot xmlns:xacro="http://www.ros.org/wiki/xacro" name="doris">
     <xacro:include filename="$(find doris_description)/urdf/doris_no_arm.urdf.xacro" />
+    <xacro:include filename="$(find hector_sensors_description)/urdf/realsense_d435_camera.urdf.xacro" />
     <joint name="dorso_arm_base" type="fixed">
         <parent link="dorso_link" />
@@ -8,3 +9,6 @@
     </joint>
     <xacro:include filename="$(find doris_arm_description)/urdf/$(arg robot_model).urdf.xacro" />
+    <!--xacro:realsense_d435_camera name="doris_arm/camera" parent="doris_arm/ee_gripper_link">
+        <origin rpy="0 0 0" xyz="-0.3 0 0.05"/>
+    </xacro:realsense_d435_camera-->
 </robot>

File: doris_description/urdf/doris_no_arm.urdf.xacro (robot description, xacro)
@@ -22,39 +22,75 @@
         <parent link="base_footprint" />
     </joint>
-    <link name="frontal_caster_link">
-        <inertial>
-            <origin xyz="0 0 0" rpy="0 0 0" />
-            <mass value="0.1" />
-            <inertia ixx="0.001" ixy="0" ixz="0" iyy="0.001" iyz="0" izz="0.001" />
-        </inertial>
-        <collision>
-            <origin xyz="0 0 0" rpy="0 0 0" />
-            <geometry>
-                <sphere radius="0.05"/>
-            </geometry>
-        </collision>
-    </link>
-    <joint name="frontal_caster_joint" type="fixed">
-        <parent link="base_link" />
-        <child link="frontal_caster_link" />
-        <origin xyz="0.2 0 0" rpy="0 0 0" />
-    </joint>
-    <link name="rear_caster_link">
-        <inertial>
-            <origin xyz="0 0 0" rpy="0 0 0" />
-            <mass value="0.1" />
-            <inertia ixx="0.001" ixy="0" ixz="0" iyy="0.001" iyz="0" izz="0.001" />
-        </inertial>
-        <collision>
-            <origin xyz="0 0 0" rpy="0 0 0" />
-            <geometry>
-                <sphere radius="0.05"/>
-            </geometry>
-        </collision>
-    </link>
-    <joint name="rear_caster_joint" type="fixed">
-        <parent link="base_link" />
-        <child link="rear_caster_link" />
-        <origin xyz="-0.2 0 0" rpy="0 0 0" />
+    <link name="frontal_left_caster_link">
+        <inertial>
+            <origin xyz="0 0 0" rpy="0 0 0" />
+            <mass value="0.1" />
+            <inertia ixx="0.001" ixy="0" ixz="0" iyy="0.001" iyz="0" izz="0.001" />
+        </inertial>
+        <collision>
+            <origin xyz="0 0 0" rpy="0 0 0" />
+            <geometry>
+                <sphere radius="0.05"/>
+            </geometry>
+        </collision>
+    </link>
+    <joint name="frontal_left_caster_joint" type="fixed">
+        <parent link="base_link" />
+        <child link="frontal_left_caster_link" />
+        <origin xyz="0.2 -0.2 0" rpy="0 0 0" />
+    </joint>
+    <link name="frontal_right_caster_link">
+        <inertial>
+            <origin xyz="0 0 0" rpy="0 0 0" />
+            <mass value="0.1" />
+            <inertia ixx="0.001" ixy="0" ixz="0" iyy="0.001" iyz="0" izz="0.001" />
+        </inertial>
+        <collision>
+            <origin xyz="0 0 0" rpy="0 0 0" />
+            <geometry>
+                <sphere radius="0.05"/>
+            </geometry>
+        </collision>
+    </link>
+    <joint name="frontal_right_caster_joint" type="fixed">
+        <parent link="base_link" />
+        <child link="frontal_right_caster_link" />
+        <origin xyz="0.2 0.2 0" rpy="0 0 0" />
+    </joint>
+    <link name="rear_left_caster_link">
+        <inertial>
+            <origin xyz="0 0 0" rpy="0 0 0" />
+            <mass value="0.1" />
+            <inertia ixx="0.001" ixy="0" ixz="0" iyy="0.001" iyz="0" izz="0.001" />
+        </inertial>
+        <collision>
+            <origin xyz="0 0 0" rpy="0 0 0" />
+            <geometry>
+                <sphere radius="0.05"/>
+            </geometry>
+        </collision>
+    </link>
+    <joint name="rear_left_caster_joint" type="fixed">
+        <parent link="base_link" />
+        <child link="rear_left_caster_link" />
+        <origin xyz="-0.2 -0.2 0" rpy="0 0 0" />
+    </joint>
+    <link name="rear_right_caster_link">
+        <inertial>
+            <origin xyz="0 0 0" rpy="0 0 0" />
+            <mass value="0.1" />
+            <inertia ixx="0.001" ixy="0" ixz="0" iyy="0.001" iyz="0" izz="0.001" />
+        </inertial>
+        <collision>
+            <origin xyz="0 0 0" rpy="0 0 0" />
+            <geometry>
+                <sphere radius="0.05"/>
+            </geometry>
+        </collision>
+    </link>
+    <joint name="rear_right_caster_joint" type="fixed">
+        <parent link="base_link" />
+        <child link="rear_right_caster_link" />
+        <origin xyz="-0.2 0.2 0" rpy="0 0 0" />
     </joint>
     <!--
@@ -155,7 +191,7 @@
             <wheelDiameter>0.2</wheelDiameter>
             <!-- Wheel acceleration, in rad/s^2, defaults to 0.0 rad/s^2 -->
-            <wheelAcceleration>1.0</wheelAcceleration>
+            <wheelAcceleration>12.6</wheelAcceleration>
             <!-- Maximum torque which the wheels can produce, in Nm, defaults to 5 Nm -->
-            <wheelTorque>200</wheelTorque>
+            <wheelTorque>400</wheelTorque>
             <!-- Topic to receive geometry_msgs/Twist message commands, defaults to `cmd_vel` -->
             <commandTopic>RosAria/cmd_vel</commandTopic>
@@ -198,12 +234,24 @@
         <mu2>0.95</mu2>
     </gazebo>
-    <gazebo reference="frontal_caster_link">
+    <gazebo reference="frontal_left_caster_link">
+        <mu1>0.000000</mu1>
+        <mu2>0.000000</mu2>
+    </gazebo>
+    <gazebo reference="frontal_right_caster_link">
+        <mu1>0.000000</mu1>
+        <mu2>0.000000</mu2>
+    </gazebo>
+    <gazebo reference="rear_left_caster_link">
+        <mu1>0.000000</mu1>
+        <mu2>0.000000</mu2>
+    </gazebo>
+    <gazebo reference="rear_right_caster_link">
+        <mu1>0.000000</mu1>
+        <mu2>0.000000</mu2>
+    </gazebo>
+    <!--gazebo reference="hokuyo_link">
         <mu1>0.000001</mu1>
         <mu2>0.000001</mu2>
-    </gazebo>
-    <gazebo reference="rear_caster_link">
-        <mu1>0.000001</mu1>
-        <mu2>0.000001</mu2>
-    </gazebo>
+    </gazebo-->
     <gazebo reference="dorso_link">
         <material>Gazebo/DarkGray</material>

File: doris_sensors_description/urdf/realsense_d435_camera.urdf.xacro (robot description, xacro)
@@ -80,5 +80,5 @@
             <sensor type="depth" name="${name}">
                 <update_rate>${update_rate}</update_rate>
-                <camera>
+                <camera name="${name}">
                     <horizontal_fov>${69.4 * M_PI/180.0}</horizontal_fov>
                     <image>
@@ -101,4 +101,6 @@
                     <frameName>${name}_${frame_name}_optical_frame</frameName>
                     <useDepth16UC1Format>true</useDepth16UC1Format>
+                    <pointCloudCutoff>${min_range}</pointCloudCutoff>
+                    <pointCloudCutoffMax>${max_range}</pointCloudCutoffMax>
                     <!-- Important information about frames: Currently, this plugin only supports simulation of color image and depth image/cloud from a single frame.
             This frame is given in the <gazebo reference=""> tag above and is set to the ${name}_link which coincides with the depth camera frame. The camera axis is the X-axis. ROS requires an optical frame
@@ -117,5 +119,5 @@
             <xacro:insert_block name="origin" />
         </xacro:realsense_d435_camera_model>
-        <xacro:realsense_d435_camera_gazebo_plugin_macro name="${name}" parent="${parent}" image_topic="image_raw" depth_points_topic="depth/points" min_range="0.3" max_range="9.0" update_rate="20"/>
+        <xacro:realsense_d435_camera_gazebo_plugin_macro name="${name}" parent="${parent}" image_topic="image_raw" depth_points_topic="depth/points" min_range="0.01" max_range="9.0" update_rate="60"/>
     </xacro:macro>
     <!--
@@ -126,5 +128,5 @@
             <xacro:insert_block name="origin" />
         </xacro:realsense_d435_camera_model_with_mount>
-        <xacro:realsense_d435_camera_gazebo_plugin_macro name="${name}" parent="${parent}" image_topic="image_raw" depth_points_topic="depth/points" min_range="0.3" max_range="9.0" update_rate="20"/>
+        <xacro:realsense_d435_camera_gazebo_plugin_macro name="${name}" parent="${parent}" image_topic="image_raw" depth_points_topic="depth/points" min_range="0.01" max_range="9.0" update_rate="60"/>
     </xacro:macro>
     <!--
@@ -136,5 +138,5 @@
             <xacro:insert_block name="origin" />
         </xacro:realsense_d435_camera_model_no_geom>
-        <xacro:realsense_camera_gazebo_plugin_macro name="${name}" parent="${parent}" image_topic="image_raw" depth_points_topic="depth/points" min_range="0.3" max_range="9.0" update_rate="20"/>
+        <xacro:realsense_camera_gazebo_plugin_macro name="${name}" parent="${parent}" image_topic="image_raw" depth_points_topic="depth/points" min_range="0.01" max_range="9.0" update_rate="60"/>
     </xacro:macro>
     <xacro:macro name="realsense_d435_camera_no_geom_comprehensive_params" params="name parent *origin image_topic depth_topic:=image_raw depth_points_topic frame_name:=color min_range max_range update_rate">
