Commit message: first commit

File: doris_sensors_description/urdf/kinect_camera.urdf.xacro (robot description, xacro)
@@ -4,8 +4,9 @@
     <xacro:property name="M_PI" value="3.1415926535897931" />
     <xacro:macro name="kinect_camera_model" params="name parent *origin">
-      <joint name="${name}_joint" type="fixed">
+      <joint name="${name}_joint" type="continuous">
         <xacro:insert_block name="origin" />
         <parent link="${parent}"/>
         <child link="${name}_link"/>
+        <axis xyz="1 0 0" />
       </joint>
       <link name="${name}_link">

Commit message: added inertial

File: doris_sensors_description/urdf/kinect_camera.urdf.xacro (robot description, xacro)
@@ -24,4 +24,11 @@
           </geometry>
         </collision>
+        <inertial>
+          <mass value = "0.170"/>
+          <origin xyz = "0 0 0"/>
+          <inertia ixx = "0.001152600" ixy = "0.0" ixz = "0.0"
+                   iyy = "0.000148934" iyz = "0.0"
+                   izz = "0.001154654"/>
+        </inertial>
       </link>
       <joint name="${name}_depth_joint" type="fixed">
@@ -43,4 +50,12 @@
       </joint>
       <link name="${name}_rgb_frame"/>
+        <inertial>
+            <mass value = "0.170"/>
+            <origin xyz = "0 0 0"/>
+            <inertia ixx = "0.001152600" ixy = "0.0" ixz = "0.0"
+                    iyy = "0.000148934" iyz = "0.0"
+                    izz = "0.001154654"/>
+        </inertial>
+      </link>
       <joint name="${name}_rgb_optical_joint" type="fixed">
         <origin xyz="0 0 0" rpy="${-M_PI/2} 0.0 ${-M_PI/2}" />

Commit message: removed intertial and added controllers

File: doris_sensors_description/urdf/kinect_camera.urdf.xacro (robot description, xacro)
@@ -24,11 +24,4 @@
           </geometry>
         </collision>
-        <inertial>
-          <mass value = "0.170"/>
-          <origin xyz = "0 0 0"/>
-          <inertia ixx = "0.001152600" ixy = "0.0" ixz = "0.0"
-                   iyy = "0.000148934" iyz = "0.0"
-                   izz = "0.001154654"/>
-        </inertial>
       </link>
       <joint name="${name}_depth_joint" type="fixed">
@@ -50,12 +43,4 @@
       </joint>
       <link name="${name}_rgb_frame"/>
-        <inertial>
-            <mass value = "0.170"/>
-            <origin xyz = "0 0 0"/>
-            <inertia ixx = "0.001152600" ixy = "0.0" ixz = "0.0"
-                    iyy = "0.000148934" iyz = "0.0"
-                    izz = "0.001154654"/>
-        </inertial>
-      </link>
       <joint name="${name}_rgb_optical_joint" type="fixed">
         <origin xyz="0 0 0" rpy="${-M_PI/2} 0.0 ${-M_PI/2}" />
@@ -85,4 +70,7 @@
             </clip>
           </camera>
+          <plugin name="gazebo_ros_control" filename="libgazebo_ros_control.so">
+            <robotNamespace>/simple_model</robotNamespace>
+          </plugin>
           <plugin name="${name}_camera_controller" filename="libgazebo_ros_openni_kinect.so">
             <imageTopicName>butia_vision/bvb/image_rgb</imageTopicName>
@@ -94,4 +82,13 @@
             <robotNamespace>/</robotNamespace>
           </plugin>
+          <transmission name="base_to_camera_trans">
+            <type>transmission_interface/SimpleTransmission</type>
+            <actuator name="motor1">
+              <mechanicalReduction>1</mechanicalReduction>
+            </actuator>
+            <joint name="camera_joint_pepe">
+              <hardwareInterface>EffortJointInterface</hardwareInterface>
+            </joint>
+          </transmission>
         </sensor>
       </gazebo>

Commit message: trying to implementing like interbotix

File: doris_sensors_description/urdf/kinect_camera.urdf.xacro (robot description, xacro)
@@ -2,8 +2,8 @@
 <robot xmlns:xacro="http://www.ros.org/wiki/xacro">
     <xacro:include filename="$(find hector_xacro_tools)/urdf/inertia_tensors.urdf.xacro"/>
-    <xacro:property name="M_PI" value="3.1415926535897931" />
+    <xacro:property name="M_PI" value="3.1415926535897931"/>
     <xacro:macro name="kinect_camera_model" params="name parent *origin">
       <joint name="${name}_joint" type="continuous">
-        <xacro:insert_block name="origin" />
+        <xacro:insert_block name="origin"/>
         <parent link="${parent}"/>
         <child link="${name}_link"/>
@@ -87,5 +87,5 @@
               <mechanicalReduction>1</mechanicalReduction>
             </actuator>
-            <joint name="camera_joint_pepe">
+            <joint name="kinect2_joint">
               <hardwareInterface>EffortJointInterface</hardwareInterface>
             </joint>
