Commit message: adding realsense in doris URDF

File: doris_sensors_description/urdf/realsense_camera.urdf.xacro (robot description, xacro)
@@ -3,4 +3,12 @@
   <xacro:property name="M_PI" value="3.1415926535897931"/>
   <xacro:macro name="realsense_camera" params="name parent *origin">
+      <!-- @TODO: GABIARRA PRA GIRAR A CAMERA -->
+      <link name="head_pan_link_static">
+          <inertial>
+              <origin rpy="0 0 0" xyz="-1.35308431126191E-16 -2.97071395261028E-17 0.0220876265081744"/>
+              <mass value="0.0182769203076134"/>
+              <inertia ixx="1.32243845065555E-05" ixy="5.07660179129181E-13" ixz="1.067515220067E-20" iyy="7.13386116649085E-06" iyz="-1.32882457845217E-20" izz="7.83291781352837E-06"/>
+          </inertial>
+      </link>
       <link name="head_pan_link">
           <inertial>
@@ -25,4 +33,11 @@
           </collision>
       </link>
+      <joint name="head_pan_joint_static" type="fixed">
+          <xacro:insert_block name="origin"/>
+          <parent link="${parent}"/>
+          <child link="head_pan_link_static"/>
+          <axis xyz="0 0 1"/>
+          <limit effort="1" lower="-1.57" upper="1.57" velocity="1"/>
+      </joint>
       <joint name="head_pan_joint" type="revolute">
           <xacro:insert_block name="origin"/>
@@ -32,4 +47,11 @@
           <limit effort="1" lower="-1.57" upper="1.57" velocity="1"/>
       </joint>
+      <link name="head_tilt_link_static">
+          <inertial>
+              <origin rpy="0 0 0" xyz="0.0168744200088311 -0.000442984145897884 -0.00405256422002387"/>
+              <mass value="0.0547677687275323"/>
+              <inertia ixx="1.07071738005716E-05" ixy="-1.46854788384565E-07" ixz="5.59529059364376E-08" iyy="1.77011620295824E-05" iyz="1.27587154712834E-09" izz="2.01583693170578E-05"/>
+          </inertial>
+      </link>
       <link name="head_tilt_link">
           <inertial>
@@ -54,4 +76,11 @@
           </collision>
       </link>
+      <joint name="head_tilt_joint_static" type="fixed">
+          <origin rpy="0 0 0" xyz="0 0 0.05"/>
+          <parent link="head_pan_link_static"/>
+          <child link="head_tilt_link_static"/>
+          <axis xyz="0 1 0"/>
+          <limit effort="1" lower="-1.57" upper="1.57" velocity="1"/>
+      </joint>
       <joint name="head_tilt_joint" type="revolute">
           <origin rpy="0 0 0" xyz="0 0 0.05"/>
@@ -61,4 +90,11 @@
           <limit effort="1" lower="-1.57" upper="1.57" velocity="1"/>
       </joint>
+      <link name="camera_link_static">
+        <inertial>
+            <origin rpy="0 0 0" xyz="-0.0132722976093535 0.00168171470080143 2.49829664994428E-06"/>
+            <mass value="0.0381925651163644"/>
+            <inertia ixx="2.4688255642946E-05" ixy="1.60697655569215E-07" ixz="1.2993241737711E-08" iyy="3.66669176935806E-06" iyz="1.30215657011203E-08" izz="2.48602467766615E-05"/>
+        </inertial>
+      </link>
       <link name="camera_link">
         <inertial>
@@ -83,4 +119,10 @@
         </collision>
       </link>
+      <joint name="camera_joint_static" type="fixed">
+          <origin rpy="0 0 0" xyz="0.06705 0 -0.00425"/>
+          <parent link="head_tilt_link_static"/>
+          <child link="camera_link_static"/>
+          <axis xyz="0 0 0"/>
+      </joint>
       <joint name="camera_joint" type="fixed">
           <origin rpy="0 0 0" xyz="0.06705 0 -0.00425"/>
