Commit message: realsense working in simulation

File: doris_sensors_description/urdf/hokuyo.urdf.xacro (robot description, xacro)
@@ -34,5 +34,5 @@
   <xacro:macro name="sim_laser_range_finder">
     <gazebo reference="hokuyo_link">
-      <sensor type="ray" name="head_hokuyo_sensor">
+      <sensor type="gpu_ray" name="head_hokuyo_sensor">
         <pose>0 0 0 0 0 0</pose>
         <visualize>false</visualize>
@@ -62,5 +62,5 @@
           </noise>
         </ray>
-        <plugin name="gazebo_ros_head_hokuyo_controller" filename="libgazebo_ros_laser.so">
+        <plugin name="gazebo_ros_head_hokuyo_controller" filename="libgazebo_ros_gpu_laser.so">
           <topicName>scan2</topicName>
           <frameName>hokuyo_link</frameName>

File: doris_sensors_description/urdf/realsense_camera.urdf.xacro (robot description, xacro)
@@ -165,4 +165,11 @@
           <origin xyz="0.06705 0 -0.00425" rpy="0 0 0"/>
       </xacro:sensor_d435> -->
+        <link name="camera_color_optical_frame" />
+        <joint name="camera_color_optical_joint" type="fixed">
+            <origin xyz="0 0 0" rpy="${-M_PI/2.0} 0 ${3*M_PI/2.0}" />
+            <!--origin xyz="0 0 0" rpy="0 0 0" /-->
+            <parent link="camera_link" />
+            <child link="camera_color_optical_frame" />
+        </joint>
   </xacro:macro>
 </robot>

File: doris_sensors_description/urdf/realsense_d435_camera.urdf.xacro (robot description, xacro)
@@ -100,4 +100,5 @@
                     <pointCloudTopicName>${depth_points_topic}</pointCloudTopicName>
                     <frameName>${name}_${frame_name}_optical_frame</frameName>
+                    <useDepth16UC1Format>true</useDepth16UC1Format>
                     <!-- Important information about frames: Currently, this plugin only supports simulation of color image and depth image/cloud from a single frame.
             This frame is given in the <gazebo reference=""> tag above and is set to the ${name}_link which coincides with the depth camera frame. The camera axis is the X-axis. ROS requires an optical frame

Commit message: changes to use two hokuyos

File: doris_sensors_description/urdf/hokuyo.urdf.xacro (robot description, xacro)
@@ -2,6 +2,6 @@
 <robot name="sensor_hokuyo"
   xmlns:xacro="http://ros.org/wiki/xacro">
-  <xacro:macro name="sensor_hokuyo" params="parent xyz rpy">
-    <link name="hokuyo_link">
+  <xacro:macro name="sensor_hokuyo" params="parent xyz rpy name">
+    <link name="hokuyo_${name}_link">
       <!--collision>
         <origin xyz="0 0 0" rpy="0 0 0"/>
@@ -22,9 +22,9 @@
       </inertial>
     </link>
-    <joint name="hokuyo_joint" type="fixed">
+    <joint name="hokuyo_${name}_joint" type="fixed">
       <!--<axis xyz="0 0 1" />-->
       <origin xyz="${xyz}" rpy="${rpy}"/>
       <parent link="${parent}"/>
-      <child link="hokuyo_link"/>
+      <child link="hokuyo_${name}_link"/>
     </joint>
     <!-- Hokuyo sensor for simulation -->
@@ -33,5 +33,5 @@
   <!-- ULM-30LX Hokuyo Laser Range Finder -->
   <xacro:macro name="sim_laser_range_finder">
-    <gazebo reference="hokuyo_link">
+    <gazebo reference="hokuyo_${name}_link">
       <sensor type="ray" name="head_hokuyo_sensor">
         <pose>0 0 0 0 0 0</pose>
@@ -64,5 +64,5 @@
         <plugin name="gazebo_ros_head_hokuyo_controller" filename="libgazebo_ros_laser.so">
           <topicName>scan2</topicName>
-          <frameName>hokuyo_link</frameName>
+          <frameName>hokuyo_${name}_link</frameName>
           <robotNamespace>/</robotNamespace>
         </plugin>
