Commit message: shark urdf working

File: shark_description/urdf/shark_description.xacro (robot description, xacro)
@@ -1,14 +1,13 @@
 <?xml version="1.0"?>
 <robot xmlns:xacro="http://www.ros.org/wiki/xacro" name="shark">
-  <xacro:property name="base_width" value="0.531"/>
-  <xacro:property name="base_len" value="0.3785"/>
-  <xacro:property name="base_height" value="0.2895"/>
-  <xacro:property name="wheel_radius" value="0.1"/>
-  <xacro:property name="base_wheel_gap" value="-0.09"/>
-  <xacro:property name="wheel_separation" value="0.35"/>
-  <xacro:property name="wheel_joint_offset" value="-0.005"/>
-  <xacro:property name="caster_height" value="0.060575"/>
-  <!-- <xacro:property name="caster_wheel_radius" value="0.0375"/>
-  <xacro:property name="caster_wheel_joint_offset" value="0.12"/> -->
+  <xacro:property name="base_width" value="0.335" />
+  <xacro:property name="base_len" value="0.5" />
+  <xacro:property name="base_height" value="0.235" />
+  <xacro:property name="wheel_radius" value="0.0825" />
+  <xacro:property name="base_wheel_gap" value="0.05" />
+  <xacro:property name="wheel_width" value="0.06" />
+  <xacro:property name="wheel_separation" value="0.39" />
+  <xacro:property name="wheel_joint_offset" value="0.0" />
+  <xacro:property name="caster_height" value="0.07" />
   <xacro:macro name="box_inertia" params="m w h d">
     <inertial>
@@ -55,8 +54,8 @@
     <link name="${prefix}_wheel">
       <visual>
-	<material name="darkgray"/>
+	      <material name="darkgray"/>
         <origin xyz="0 0 0" rpy="${pi/2} 0 0"/>
         <geometry>
-          <cylinder radius="${wheel_radius}" length="0.05"/>
+          <cylinder radius="${wheel_radius}" length="${wheel_width}"/>
         </geometry>
       </visual>
