Commit message: :wrench: updated wheel radius and minor changes

File: shark_description/urdf/shark.xacro (robot description, xacro)
@@ -1,5 +1,5 @@
 <?xml version="1.0"?>
 <!-- Basic differential drive mobile base -->
-<robot xmlns:xacro="http://www.ros.org/wiki/xacro" name="shark_mb">
+<robot xmlns:xacro="http://www.ros.org/wiki/xacro" name="shark">
   <xacro:include filename="$(find shark_description)/urdf/shark_description.xacro" />
   <!-- Import Rviz colors -->

File: shark_description/urdf/shark_description.xacro (robot description, xacro)
@@ -1,8 +1,8 @@
 <?xml version="1.0"?>
-<robot xmlns:xacro="http://www.ros.org/wiki/xacro" name="shark">
+<robot xmlns:xacro="http://www.ros.org/wiki/xacro" name="shark_description">
   <xacro:property name="base_width" value="0.335" />
   <xacro:property name="base_len" value="0.5" />
   <xacro:property name="base_height" value="0.235" />
-  <xacro:property name="wheel_radius" value="0.0825" />
+  <xacro:property name="wheel_radius" value="0.055" />
   <xacro:property name="base_wheel_gap" value="0.05" />
   <xacro:property name="wheel_width" value="0.06" />
@@ -105,4 +105,3 @@
     <origin xyz="${caster_wheel_joint_offset} 0 -${0.06+caster_wheel_radius}" rpy="0 0 0"/>
   </joint> -->
-  <!-- <xacro:sensor_hokuyo parent="base_link" xyz="${base_len/2 + 0.025 + 0.0159} 0 ${0.02 - base_height/2}" rpy="0 0 0" name="ground" /> -->
 </robot>
