Commit message: :arrow_up: added urg_node as dependencie

File: logistic_description/urdf/logistic.xacro (robot description, xacro)
@@ -11,3 +11,5 @@
         <origin xyz="${base_len/2 - 0.07} 0 ${base_height/2}" rpy="0 0 0" />
     </xacro:VLP-16>
+    <xacro:include filename="$(find sensors_description)/urdf/hokuyo.xacro" />
+    <xacro:sensor_hokuyo parent="base_link" xyz="${base_len/2 + 0.017 + 0.024} 0 ${0.02 - base_height/2}" rpy="3.14 0 0" name="ground"/>
 </robot>

File: sensors_description/urdf/hokuyo.xacro (robot description, xacro)
@@ -13,5 +13,5 @@
         <origin xyz="0 0 0" rpy="0 0 0"/>
         <geometry>
-          <mesh filename="package://doris_sensors_description/meshes/sensors/hokuyo.dae"/>
+          <mesh filename="package://sensors_description/meshes/hokuyo.dae"/>
         </geometry>
       </visual>

Commit message: :bug: fixed wheel radius

File: logistic_description/urdf/logistic.xacro (robot description, xacro)
@@ -13,3 +13,12 @@
     <xacro:include filename="$(find sensors_description)/urdf/hokuyo.xacro" />
     <xacro:sensor_hokuyo parent="base_link" xyz="${base_len/2 + 0.017 + 0.024} 0 ${0.02 - base_height/2}" rpy="3.14 0 0" name="ground"/>
+    <xacro:macro name="imu" params="parent xyz rpy">
+    <link name="imu_link"/>
+    <joint name="imu_joint" type="fixed">
+      <parent link="${parent}"/>
+      <child link="imu_link"/>
+      <origin xyz="${xyz}" rpy="${rpy}"/>
+    </joint>
+    </xacro:macro>
+    <xacro:imu parent="base_link" xyz="${base_len/2 + 0.0625} 0 ${0.02 - base_height/2}" rpy="0 0 0"/>
 </robot>

File: shark_description/ros2_control/shark_ros2_control.xacro (robot description, xacro)
@@ -4,7 +4,7 @@
     <hardware>
       <plugin>hoverboard_driver/hoverboard_driver</plugin>
-      <param name="wheel_radius">0.055</param>
+      <param name="wheel_radius">0.0775</param>
       <param name="max_velocity">1.0</param>
-      <param name="device">/dev/ttyUSB0</param>
+      <param name="device">/dev/ttyUSB1</param>
     </hardware>
     <joint name="left_wheel_joint">

File: shark_description/urdf/shark_description.xacro (robot description, xacro)
@@ -4,8 +4,8 @@
   <xacro:property name="base_len" value="0.5" />
   <xacro:property name="base_height" value="0.235" />
-  <xacro:property name="wheel_radius" value="0.055" />
+  <xacro:property name="wheel_radius" value="0.0775" />
   <xacro:property name="base_wheel_gap" value="0.05" />
   <xacro:property name="wheel_width" value="0.06" />
-  <xacro:property name="wheel_separation" value="0.39" />
+  <xacro:property name="wheel_separation" value="0.41" />
   <xacro:property name="wheel_joint_offset" value="0.0" />
   <xacro:property name="caster_height" value="0.07" />
